File: LED HIGH SIDE DRIVER.sch (KiCad schematic (older format))
At the start: 70 parts

Commit message: 8-24
Started separating out the power supply and building the PCB
Parts:
- removed P? (x2): CONN_8, symbol CONN_8
- removed P?: CONN_5, symbol CONN_5
- removed P?: CONN_2, symbol CONN_2
- removed Q? (x8): NPN, ~, symbol NPN
- removed Q? (x8): MOSFET_N, ~, symbol MOSFET_N
- removed R? (x7): 10K, ~, symbol R
- removed R? (x5): 1K, ~, symbol R
- added P10, P9: CONN_8, symbol CONN_8
- added P7: CONN_2, symbol CONN_2
- added P8: CONN_5, symbol CONN_5
- added Q37, Q39, Q49, Q50, Q52, Q54, Q55, Q56: NPN, ~, symbol NPN
- added Q43, Q44, Q45, Q46, Q47, Q58, Q60, Q64: MOSFET_N, ~, symbol MOSFET_N
- added R33, R36, R37, R38, R42: 1K, ~, symbol R
- added R53, R54, R59, R60, R62, R63, R64: 10K, ~, symbol R
- gave numbers to parts that had none: 38
Connections:
- net 12V: now also P7.1 (P1), R53.1, R54.1, R59.1, R60.1, R62.1, R63.1, R64.1
- net CLK: now also P8.2
- net DATA_IN: now also P8.1
- net GND: now also P7.2 (PM), P8.5, Q37.1 (E), Q39.1 (E), Q43.S, Q44.S, Q45.S, Q46.S, Q47.S, Q49.1 (E), Q50.1 (E), Q52.1 (E), Q54.1 (E), Q55.1 (E), Q56.1 (E), Q58.S, Q60.S, Q64.S
- net LATCH: now also P8.3
- net SINK1: now also P9.1 (P1)
- net SINK10: now also P10.2 (P2)
- net SINK11: now also P10.3 (P3), Q46.D
- net SINK12: now also P10.4 (P4)
- net SINK13: now also P10.5 (P5), Q47.D
- net SINK14: now also P10.6 (P6)
- net SINK15: now also P10.7 (P7)
- net SINK16: now also P10.8 (P8), Q64.D
- net SINK2: now also P9.2 (P2)
- net SINK3: now also P9.3 (P3)
- net SINK4: now also P9.4 (P4), Q58.D
- net SINK5: now also P9.5 (P5), Q43.D
- net SINK6: now also P9.6 (P6)
- net SINK7: now also P9.7 (P7), Q44.D
- net SINK8: now also P9.8 (P8), Q60.D
- net SINK9: now also P10.1 (P1), Q45.D
- net VCC3.3: now also P8.4
- net at U6.15 (QA): now also R33.2
- net at U6.2 (QC): now also R37.2
- net at U6.3 (QD): now also R38.2
- net at U6.7 (QH): now also R42.2
- net at Q33.2 (B): now also R33.1
- net at Q57.G, R57.2: now also Q49.3 (C)
- net at R34.1: now also Q49.2 (B)
- net at Q34.2 (B): now also R37.1
- net at R58.2: now also Q50.3 (C), Q58.G
- net at Q35.3 (C), R51.2: now also Q43.G
- net at Q51.3 (C), Q59.G: now also R59.2
- net at Q36.3 (C), R52.2: now also Q44.G
- net at U7.1 (QB): now also R36.2
- net at R35.1: now also Q37.2 (B)
- net at Q53.2 (B): now also R36.1
- net at Q38.3 (C): now also Q46.G, R54.2
- net at Q62.G: now also Q54.3 (C), R62.2
- net at R44.1: now also Q54.2 (B)
- net at R55.2: now also Q39.3 (C), Q47.G
- net at R45.1: now also Q39.2 (B)
- net at Q63.G: now also Q55.3 (C), R63.2
- net at R46.1: now also Q55.2 (B)
- net at R48.1: now also Q56.2 (B)
- new net: Q50.2 (B), R38.1
- new net: Q52.3 (C), Q60.G, R60.2
- new net: Q52.2 (B), R42.1
- new net: Q37.3 (C), Q45.G, R53.2
- new net: Q56.3 (C), Q64.G, R64.2
