File: LED LOW SIDE DRIVER.sch (KiCad schematic (older format))
At the start: 70 parts

Commit message: 8-24
Started separating out the power supply and building the PCB
Parts:
- removed Q? (x8): NPN, ~, symbol NPN
- removed Q? (x8): MOSFET_N, ~, symbol MOSFET_N
- removed R? (x9): 10K, ~, symbol R
- removed R? (x11): 1K, ~, symbol R
- removed U? (x2): 74HC595, ~, symbol 74HC595
- added Q1, Q19, Q2, Q21, Q3, Q4, Q6, Q8: NPN, ~, symbol NPN
- added Q10, Q16, Q25, Q27, Q29, Q30, Q31, Q9: MOSFET_N, ~, symbol MOSFET_N
- added R11, R12, R13, R14, R15, R16, R2, R3, R7, R8, R9: 1K, ~, symbol R
- added R17, R18, R19, R20, R23, R24, R25, R26, R29: 10K, ~, symbol R
- added U4, U5: 74HC595, ~, symbol 74HC595
- gave numbers to parts that had none: 32
Connections:
- net 12V: now also R17.1, R18.1, R19.1, R20.1, R23.1, R24.1, R25.1, R26.1, R29.1
- net CLOCK: now also U4.11 (SRCLK), U5.11 (SRCLK)
- net DATA_IN: now also U4.14 (SER)
- net DATA_OUT: now also U5.9 (~QH)
- net GND: now also Q1.1 (E), Q10.S, Q16.S, Q19.1 (E), Q2.1 (E), Q21.1 (E), Q25.S, Q27.S, Q29.S, Q3.1 (E), Q30.S, Q31.S, Q4.1 (E), Q6.1 (E), Q8.1 (E), Q9.S, U4.13 (G), U4.8 (GND), U5.13 (G), U5.8 (GND)
- net LATCH: now also U4.12 (RCLK), U5.12 (RCLK)
- net SINK1: now also Q9.D
- net SINK10: now also Q29.D
- net SINK12: now also Q30.D
- net SINK14: now also Q31.D
- net SINK15: now also Q16.D
- net SINK2: now also Q25.D
- net SINK3: now also Q10.D
- net SINK6: now also Q27.D
- net VCC: now also U4.16 (VCC), U5.16 (VCC)
- net VDD3.3: now also U4.10 (SRCLR), U5.10 (SRCLR)
- net at R1.2: now also U4.15 (QA)
- net at R5.2: now also U4.2 (QC)
- net at R6.2: now also U4.3 (QD)
- net at R10.2: now also U4.7 (QH)
- net at R1.1: now also Q1.2 (B)
- net at Q17.3 (C): now also Q25.G, R25.2
- net at Q17.2 (B): now also R2.1
- net at R5.1: now also Q2.2 (B)
- net at Q18.3 (C), Q26.G: now also R26.2
- net at Q11.G: now also Q3.3 (C), R19.2
- net at R27.2: now also Q19.3 (C), Q27.G
- net at Q12.G: now also Q4.3 (C), R20.2
- net at R4.2: now also U5.1 (QB)
- net at Q5.2 (B): now also R3.1
- net at R4.1: now also Q21.2 (B)
- net at Q14.G, R22.2: now also Q6.3 (C)
- net at Q22.3 (C), R30.2: now also Q30.G
- net at Q22.2 (B): now also R12.1
- net at Q15.G, Q7.3 (C): now also R23.2
- net at Q7.2 (B): now also R13.1
- net at Q23.3 (C), R31.2: now also Q31.G
- net at Q23.2 (B): now also R14.1
- net at Q24.2 (B): now also R16.1
- new net: R2.2, U4.1 (QB)
- new net: R7.2, U4.4 (QE)
- new net: R8.2, U4.5 (QF)
- new net: R9.2, U4.6 (QG)
- new net: U4.9 (~QH), U5.14 (SER)
- new net: Q1.3 (C), Q9.G, R17.2
- new net: Q10.G, Q2.3 (C), R18.2
- new net: Q3.2 (B), R7.1
- new net: Q19.2 (B), R8.1
- new net: Q4.2 (B), R9.1
- new net: R3.2, U5.15 (QA)
- new net: R11.2, U5.2 (QC)
- new net: R12.2, U5.3 (QD)
- new net: R13.2, U5.4 (QE)
- new net: R14.2, U5.5 (QF)
- new net: R15.2, U5.6 (QG)
- new net: R16.2, U5.7 (QH)
- new net: Q21.3 (C), Q29.G, R29.2
- new net: Q6.2 (B), R11.1
- new net: Q16.G, Q8.3 (C), R24.2
- new net: Q8.2 (B), R15.1
