File: Scoreboard.sch (KiCad schematic (older format))
At the start: 0 parts

Commit message: 8-24
Started separating out the power supply and building the PCB
Changed lines of the file:
@@
 LIBS:WF121
 LIBS:CustomPower
+LIBS:CustomConnect
 LIBS:Scoreboard-cache
 EELAYER 27 0
@@
 Sheet 1 5
 Title ""
-Date "23 aug 2014"
+Date "24 aug 2014"
 Rev ""
 Comp ""
@@
 F42 "RD10" B L 6850 6050 60
 $EndSheet
-Wire Wire Line
-	10200 4100 9750 4100
-Wire Wire Line
-	9750 4100 9750 6050
-Wire Wire Line
-	9750 6050 8400 6050
 $Sheet
 S 2000 3750 1300 2800
