File: WIFI_Controller.sch (KiCad schematic (older format))
At the start: 5 parts

Commit message: 8-24
Started separating out the power supply and building the PCB
Parts:
- gave numbers to parts that had none: 5
Changed lines of the file:
@@
 LIBS:WF121
 LIBS:CustomPower
+LIBS:CustomConnect
 LIBS:Scoreboard-cache
 EELAYER 27 0
@@
 Sheet 3 5
 Title ""
-Date "23 aug 2014"
+Date "24 aug 2014"
 Rev ""
 Comp ""
@@
 $EndDescr
 $Comp
-L WF121 MOD?
+L WF121 MOD1
 U 1 1 53F54C1F
 P 4850 3150
-F 0 "MOD?" H 6700 2730 50  0000 L BNN
+F 0 "MOD1" H 6700 2730 50  0000 L BNN
 F 1 "WF121" H 5550 2350 50  0000 L BNN
 F 2 "DIP8" H 4450 2750 50  0001 C CNN
@@
 $EndComp
 $Comp
-L GND #PWR?
+L GND #PWR011
 U 1 1 53F54C25
 P 4600 2100
-F 0 "#PWR?" H 4600 2100 30  0001 C CNN
+F 0 "#PWR011" H 4600 2100 30  0001 C CNN
 F 1 "GND" H 4600 2030 30  0001 C CNN
 F 2 "" H 4600 2100 60  0000 C CNN
@@
 $EndComp
 $Comp
-L GND #PWR?
+L GND #PWR012
 U 1 1 53F54C2F
 P 6500 3850
-F 0 "#PWR?" H 6500 3850 30  0001 C CNN
+F 0 "#PWR012" H 6500 3850 30  0001 C CNN
 F 1 "GND" H 6500 3780 30  0001 C CNN
 F 2 "" H 6500 3850 60  0000 C CNN
@@
 $EndComp
 $Comp
-L GND #PWR?
+L GND #PWR013
 U 1 1 53F54C35
 P 6500 2050
-F 0 "#PWR?" H 6500 2050 30  0001 C CNN
+F 0 "#PWR013" H 6500 2050 30  0001 C CNN
 F 1 "GND" H 6500 1980 30  0001 C CNN
 F 2 "" H 6500 2050 60  0000 C CNN
@@
 $EndComp
 $Comp
-L GND #PWR?
+L GND #PWR014
 U 1 1 53F54C3B
 P 5000 3900
-F 0 "#PWR?" H 5000 3900 30  0001 C CNN
+F 0 "#PWR014" H 5000 3900 30  0001 C CNN
 F 1 "GND" H 5000 3830 30  0001 C CNN
 F 2 "" H 5000 3900 60  0000 C CNN
@@
 $EndComp
 $Comp
-L GND #PWR?
+L GND #PWR015
 U 1 1 53F54C41
 P 3950 2950
-F 0 "#PWR?" H 3950 2950 30  0001 C CNN
+F 0 "#PWR015" H 3950 2950 30  0001 C CNN
 F 1 "GND" H 3950 2880 30  0001 C CNN
 F 2 "" H 3950 2950 60  0000 C CNN
@@
 $EndComp
 $Comp
-L GND #PWR?
+L GND #PWR016
 U 1 1 53F54C47
 P 3950 2750
-F 0 "#PWR?" H 3950 2750 30  0001 C CNN
+F 0 "#PWR016" H 3950 2750 30  0001 C CNN
 F 1 "GND" H 3950 2680 30  0001 C CNN
 F 2 "" H 3950 2750 60  0000 C CNN
@@
 $EndComp
 $Comp
-L GND #PWR?
+L GND #PWR017
 U 1 1 53F54C4D
 P 4400 3900
-F 0 "#PWR?" H 4400 3900 30  0001 C CNN
+F 0 "#PWR017" H 4400 3900 30  0001 C CNN
 F 1 "GND" H 4400 3830 30  0001 C CNN
 F 2 "" H 4400 3900 60  0000 C CNN
@@
 $EndComp
 $Comp
-L CONN_6 P?
+L CONN_6 P1
 U 1 1 53F54C62
 P 2550 2550
-F 0 "P?" V 2500 2550 60  0000 C CNN
+F 0 "P1" V 2500 2550 60  0000 C CNN
 F 1 "PicKit3 Header 1X6" V 2600 2550 60  0000 C CNN
 F 2 "" H 2550 2550 60  0000 C CNN
@@
 $EndComp
 $Comp
-L C C?
+L C C5
 U 1 1 53F54C6A
 P 5500 4400
-F 0 "C?" H 5500 4500 40  0000 L CNN
+F 0 "C5" H 5500 4500 40  0000 L CNN
 F 1 "C" H 5506 4315 40  0000 L CNN
 F 2 "~" H 5538 4250 30  0000 C CNN
@@
 $EndComp
 $Comp
-L C C?
+L C C6
 U 1 1 53F54C70
 P 6000 4400
-F 0 "C?" H 6000 4500 40  0000 L CNN
+F 0 "C6" H 6000 4500 40  0000 L CNN
 F 1 "C" H 6006 4315 40  0000 L CNN
 F 2 "~" H 6038 4250 30  0000 C CNN
@@
 $EndComp
 $Comp
-L GND #PWR?
+L GND #PWR018
 U 1 1 53F54C76
 P 6000 4600
-F 0 "#PWR?" H 6000 4600 30  0001 C CNN
+F 0 "#PWR018" H 6000 4600 30  0001 C CNN
 F 1 "GND" H 6000 4530 30  0001 C CNN
 F 2 "" H 6000 4600 60  0000 C CNN
@@
 $EndComp
 $Comp
-L GND #PWR?
+L GND #PWR019
 U 1 1 53F54C7C
 P 5500 4600
-F 0 "#PWR?" H 5500 4600 30  0001 C CNN
+F 0 "#PWR019" H 5500 4600 30  0001 C CNN
 F 1 "GND" H 5500 4530 30  0001 C CNN
 F 2 "" H 5500 4600 60  0000 C CNN
@@
 $EndComp
 $Comp
-L GND #PWR?
+L GND #PWR020
 U 1 1 53F54C84
 P 1900 2500
-F 0 "#PWR?" H 1900 2500 30  0001 C CNN
+F 0 "#PWR020" H 1900 2500 30  0001 C CNN
 F 1 "GND" H 1900 2430 30  0001 C CNN
 F 2 "" H 1900 2500 60  0000 C CNN
@@
 	7350 3050 7000 3050
 $Comp
-L CONN_10X2 P?
+L CONN_10X2 P2
 U 1 1 53F54DDE
 P 2550 4800
-F 0 "P?" H 2550 5350 60  0000 C CNN
+F 0 "P2" H 2550 5350 60  0000 C CNN
 F 1 "CONN_10X2_JTAG" V 2550 4700 50  0000 C CNN
 F 2 "" H 2550 4800 60  0000 C CNN
@@
 Connection ~ 2950 5150
 $Comp
-L GND #PWR?
+L GND #PWR021
 U 1 1 53F54F44
 P 2950 5500
-F 0 "#PWR?" H 2950 5500 30  0001 C CNN
+F 0 "#PWR021" H 2950 5500 30  0001 C CNN
 F 1 "GND" H 2950 5430 30  0001 C CNN
 F 2 "" H 2950 5500 60  0000 C CNN
