File: PowerSupply/$Scoreboard_PowerSupply.sch (KiCad schematic (older format))
At the start: 11 parts, among them CON1 12V INPUT, U1 MCP16321/2, U2 12V OUT, U3 3.3V OUT

Commit message: 8-24
Started separating out the power supply and building the PCB
Parts:
- removed C1, C4: 100uF, ~, symbol C
- removed U1: MCP16321/2, ~, symbol MCP16321/2
- removed U3: 3.3V OUT, symbol WIRE2
- added C1, C4: 100uF, ~, symbol CP1
- added C5: 4.7uF, ~, symbol C
- added U1, U4: 12V OUT, symbol WIRE2
- added U3: MCP16321/2, ~, symbol MCP16321/2
- added U5: 3.3V OUT, symbol WIRE2
- C2: value 20uF -> 4.7uF
- F1: value 20A -> 7A
- U2: value 12V OUT -> 3.3V OUT
Connections:
- net 12V: now also C1.1, C5.1, U1.1, U3.2 (VIN), U4.1; no longer U2.1
- net 3.3V: now also U2.1, C4.1, U3.5 (FB), U5.1
- net GND: now also C1.2, C4.2, C5.2, U1.2, U3.15 (PGND), U3.17 (EP), U3.4 (SGND), U4.2, U5.2
- net at C3.1: now also U3.10 (BOOST)
- net at L1.2: now also U3.12 (SW)
Changed lines of the file:
@@
 LIBS:contrib
 LIBS:valves
-LIBS:WF121
+LIBS:CustomConnect
 LIBS:CustomPower
-LIBS:CustomConnect
-LIBS:Scoreboard-cache
+LIBS:Scoreboard_PowerSupply-cache
 EELAYER 27 0
 EELAYER END
 $Descr A4 11693 8268
 encoding utf-8
-Sheet 2 5
+Sheet 1 1
 Title ""
 Date "24 aug 2014"
@@
 $Comp
 L BARREL_JACK CON1
-U 1 1 53F54474
+U 1 1 53FA573E
 P 2900 3600
 F 0 "CON1" H 2900 3850 60  0000 C CNN
@@
 $Comp
 L GND #PWR01
-U 1 1 53F5447A
+U 1 1 53FA573F
 P 3400 3950
 F 0 "#PWR01" H 3400 3950 30  0001 C CNN
@@
 $EndComp
 $Comp
-L MCP16321/2 U1
-U 1 1 53F54480
+L MCP16321/2 U3
+U 1 1 53FA5740
 P 6200 4200
-F 0 "U1" H 6200 4200 60  0000 C CNN
+F 0 "U3" H 6200 4200 60  0000 C CNN
 F 1 "MCP16321/2" H 5900 4300 60  0000 C CNN
 F 2 "~" H 6200 4200 60  0000 C CNN
@@
 $Comp
 L GND #PWR02
-U 1 1 53F54486
+U 1 1 53FA5741
 P 4450 4300
 F 0 "#PWR02" H 4450 4300 30  0001 C CNN
@@
 $Comp
 L FUSE F1
-U 1 1 53F5448C
+U 1 1 53FA5742
 P 3750 3500
 F 0 "F1" H 3850 3550 40  0000 C CNN
-F 1 "20A" H 3650 3450 40  0000 C CNN
+F 1 "7A" H 3650 3450 40  0000 C CNN
 F 2 "~" H 3750 3500 60  0000 C CNN
 F 3 "~" H 3750 3500 60  0000 C CNN
@@
 $EndComp
 $Comp
-L C C1
-U 1 1 53F54492
-P 4450 3900
-F 0 "C1" H 4450 4000 40  0000 L CNN
-F 1 "100uF" H 4456 3815 40  0000 L CNN
-F 2 "~" H 4488 3750 30  0000 C CNN
-F 3 "~" H 4450 3900 60  0000 C CNN
-	1    4450 3900
-	1    0    0    -1
-$EndComp
-$Comp
 L DIODE D1
-U 1 1 53F54498
+U 1 1 53FA5744
 P 4150 3900
 F 0 "D1" H 4150 4000 40  0000 C CNN
@@
 $Comp
 L GND #PWR03
-U 1 1 53F5449E
+U 1 1 53FA5745
 P 4150 4300
 F 0 "#PWR03" H 4150 4300 30  0001 C CNN
@@
 $Comp
 L GND #PWR04
-U 1 1 53F544AE
+U 1 1 53FA5746
 P 6450 4500
 F 0 "#PWR04" H 6450 4500 30  0001 C CNN
@@
 $Comp
 L GND #PWR05
-U 1 1 53F544B4
+U 1 1 53FA5747
 P 6700 4500
 F 0 "#PWR05" H 6700 4500 30  0001 C CNN
@@
 $Comp
 L C C3
-U 1 1 53F545A8
+U 1 1 53FA5748
 P 7050 3050
 F 0 "C3" H 7050 3150 40  0000 L CNN
@@
 $Comp
 L INDUCTOR L1
-U 1 1 53F545EA
+U 1 1 53FA5749
 P 7550 3550
 F 0 "L1" V 7500 3550 40  0000 C CNN
@@
 3.3V
 $Comp
-L C C4
-U 1 1 53F54818
-P 8300 3850
-F 0 "C4" H 8300 3950 40  0000 L CNN
-F 1 "100uF" H 8306 3765 40  0000 L CNN
-F 2 "~" H 8338 3700 30  0000 C CNN
-F 3 "~" H 8300 3850 60  0000 C CNN
-	1    8300 3850
-	1    0    0    -1
-$EndComp
-$Comp
 L GND #PWR06
-U 1 1 53F5484A
+U 1 1 53FA574B
 P 8300 4200
 F 0 "#PWR06" H 8300 4200 30  0001 C CNN
@@
 $Comp
 L C C2
-U 1 1 53F5487E
+U 1 1 53FA574C
 P 5400 3850
 F 0 "C2" H 5400 3950 40  0000 L CNN
-F 1 "20uF" H 5406 3765 40  0000 L CNN
+F 1 "4.7uF" H 5406 3765 40  0000 L CNN
 F 2 "~" H 5438 3700 30  0000 C CNN
 F 3 "~" H 5400 3850 60  0000 C CNN
@@
 $Comp
 L GND #PWR07
-U 1 1 53F54892
+U 1 1 53FA574D
 P 5400 4200
 F 0 "#PWR07" H 5400 4200 30  0001 C CNN
@@
 $Comp
 L GND #PWR08
-U 1 1 53F548DB
+U 1 1 53FA574E
 P 5850 4500
 F 0 "#PWR08" H 5850 4500 30  0001 C CNN
@@
 $EndComp
 $Comp
+L WIRE2 U1
+U 1 1 53FA574F
+P 5800 5950
+F 0 "U1" H 5800 5950 60  0000 C CNN
+F 1 "12V OUT" H 5800 6800 60  0000 C CNN
+F 2 "" H 5800 5950 60  0000 C CNN
+F 3 "" H 5800 5950 60  0000 C CNN
+	1    5800 5950
+	1    0    0    -1
+$EndComp
+$Comp
 L WIRE2 U2
-U 1 1 53FA48BE
-P 3950 6050
-F 0 "U2" H 3950 6050 60  0000 C CNN
-F 1 "12V OUT" H 3950 6900 60  0000 C CNN
-F 2 "" H 3950 6050 60  0000 C CNN
-F 3 "" H 3950 6050 60  0000 C CNN
-	1    3950 6050
-	1    0    0    -1
-$EndComp
-$Comp
-L WIRE2 U3
-U 1 1 53FA48CD
-P 5600 6050
-F 0 "U3" H 5600 6050 60  0000 C CNN
-F 1 "3.3V OUT" H 5600 6900 60  0000 C CNN
-F 2 "" H 5600 6050 60  0000 C CNN
-F 3 "" H 5600 6050 60  0000 C CNN
-	1    5600 6050
+U 1 1 53FA5750
+P 7450 5950
+F 0 "U2" H 7450 5950 60  0000 C CNN
+F 1 "3.3V OUT" H 7450 6800 60  0000 C CNN
+F 2 "" H 7450 5950 60  0000 C CNN
+F 3 "" H 7450 5950 60  0000 C CNN
+	1    7450 5950
 	1    0    0    -1
 $EndComp
 $Comp
 L GND #PWR09
-U 1 1 53FA48FA
-P 4950 5900
-F 0 "#PWR09" H 4950 5900 30  0001 C CNN
-F 1 "GND" H 4950 5830 30  0001 C CNN
-F 2 "" H 4950 5900 60  0000 C CNN
-F 3 "" H 4950 5900 60  0000 C CNN
-	1    4950 5900
+U 1 1 53FA5751
+P 6800 5800
+F 0 "#PWR09" H 6800 5800 30  0001 C CNN
+F 1 "GND" H 6800 5730 30  0001 C CNN
+F 2 "" H 6800 5800 60  0000 C CNN
+F 3 "" H 6800 5800 60  0000 C CNN
+	1    6800 5800
 	1    0    0    -1
 $EndComp
 $Comp
 L GND #PWR010
-U 1 1 53FA4909
-P 3250 5900
-F 0 "#PWR010" H 3250 5900 30  0001 C CNN
-F 1 "GND" H 3250 5830 30  0001 C CNN
-F 2 "" H 3250 5900 60  0000 C CNN
-F 3 "" H 3250 5900 60  0000 C CNN
-	1    3250 5900
-	1    0    0    -1
-$EndComp
-Text HLabel 4950 5450 0    39   Output ~ 0
+U 1 1 53FA5752
+P 5100 5800
+F 0 "#PWR010" H 5100 5800 30  0001 C CNN
+F 1 "GND" H 5100 5730 30  0001 C CNN
+F 2 "" H 5100 5800 60  0000 C CNN
+F 3 "" H 5100 5800 60  0000 C CNN
+	1    5100 5800
+	1    0    0    -1
+$EndComp
+Text HLabel 6800 5350 0    39   Output ~ 0
 3.3V
-Text HLabel 3300 5450 0    39   Output ~ 0
+Text HLabel 5150 5350 0    39   Output ~ 0
 12V
-Text HLabel 5250 3100 1    39   Input ~ 0
+Text HLabel 4750 3100 1    39   Input ~ 0
 12V
 Wire Wire Line
@@
 	6700 4300 6700 4500
 Wire Wire Line
-	5250 3100 5250 3500
-Connection ~ 5250 3500
+	4750 3100 4750 3500
+Connection ~ 4750 3500
 Wire Wire Line
 	7000 3550 7250 3550
@@
 	5850 3900 5850 4500
 Wire Wire Line
-	4950 5750 5100 5750
-Wire Wire Line
-	4950 5750 4950 5900
-Wire Wire Line
-	3450 5750 3250 5750
-Wire Wire Line
-	3250 5750 3250 5900
-Wire Wire Line
-	5100 5450 4950 5450
-Wire Wire Line
-	3450 5450 3300 5450
+	6800 5650 6950 5650
+Wire Wire Line
+	6800 5650 6800 5800
+Wire Wire Line
+	5300 5650 5100 5650
+Wire Wire Line
+	5100 5650 5100 5800
+Wire Wire Line
+	6950 5350 6800 5350
+Wire Wire Line
+	5300 5350 5150 5350
+$Comp
+L WIRE2 U5
+U 1 1 53FA57F1
+P 8750 5950
+F 0 "U5" H 8750 5950 60  0000 C CNN
+F 1 "3.3V OUT" H 8750 6800 60  0000 C CNN
+F 2 "" H 8750 5950 60  0000 C CNN
+F 3 "" H 8750 5950 60  0000 C CNN
+	1    8750 5950
+	1    0    0    -1
+$EndComp
+$Comp
+L WIRE2 U4
+U 1 1 53FA57F7
+P 4350 5950
+F 0 "U4" H 4350 5950 60  0000 C CNN
+F 1 "12V OUT" H 4350 6800 60  0000 C CNN
+F 2 "" H 4350 5950 60  0000 C CNN
+F 3 "" H 4350 5950 60  0000 C CNN
+	1    4350 5950
+	1    0    0    -1
+$EndComp
+$Comp
+L GND #PWR011
+U 1 1 53FA57FF
+P 8100 5850
+F 0 "#PWR011" H 8100 5850 30  0001 C CNN
+F 1 "GND" H 8100 5780 30  0001 C CNN
+F 2 "" H 8100 5850 60  0000 C CNN
+F 3 "" H 8100 5850 60  0000 C CNN
+	1    8100 5850
+	1    0    0    -1
+$EndComp
+$Comp
+L GND #PWR012
+U 1 1 53FA580E
+P 3600 5800
+F 0 "#PWR012" H 3600 5800 30  0001 C CNN
+F 1 "GND" H 3600 5730 30  0001 C CNN
+F 2 "" H 3600 5800 60  0000 C CNN
+F 3 "" H 3600 5800 60  0000 C CNN
+	1    3600 5800
+	1    0    0    -1
+$EndComp
+Text HLabel 3550 5350 0    39   Output ~ 0
+12V
+Text HLabel 8000 5350 0    39   Output ~ 0
+3.3V
+Wire Wire Line
+	8250 5350 8000 5350
+Wire Wire Line
+	3850 5350 3550 5350
+Wire Wire Line
+	3850 5650 3600 5650
+Wire Wire Line
+	3600 5650 3600 5800
+Wire Wire Line
+	8250 5650 8100 5650
+Wire Wire Line
+	8100 5650 8100 5850
+$Comp
+L CP1 C4
+U 1 1 53FA59E2
+P 8300 3850
+F 0 "C4" H 8350 3950 50  0000 L CNN
+F 1 "100uF" H 8350 3750 50  0000 L CNN
+F 2 "~" H 8300 3850 60  0000 C CNN
+F 3 "~" H 8300 3850 60  0000 C CNN
+	1    8300 3850
+	1    0    0    -1
+$EndComp
+$Comp
+L CP1 C1
+U 1 1 53FA59F1
+P 4450 3900
+F 0 "C1" H 4500 4000 50  0000 L CNN
+F 1 "100uF" H 4500 3800 50  0000 L CNN
+F 2 "~" H 4450 3900 60  0000 C CNN
+F 3 "~" H 4450 3900 60  0000 C CNN
+	1    4450 3900
+	1    0    0    -1
+$EndComp
+$Comp
+L C C5
+U 1 1 53FA61A3
+P 5150 3850
+F 0 "C5" H 5150 3950 40  0000 L CNN
+F 1 "4.7uF" H 5156 3765 40  0000 L CNN
+F 2 "~" H 5188 3700 30  0000 C CNN
+F 3 "~" H 5150 3850 60  0000 C CNN
+	1    5150 3850
+	1    0    0    -1
+$EndComp
+Wire Wire Line
+	5150 3650 5150 3500
+Connection ~ 5150 3500
+Wire Wire Line
+	5150 4050 5400 4050
 $EndSCHEMATC
