File: PowerSupply/Scoreboard_PowerSupply.sch (KiCad schematic (older format))
At the start: 11 parts, among them CON1 12V INPUT, U1 MCP16321/2, U2 12V OUT, U3 3.3V OUT

Commit message: 8-24
Started separating out the power supply and building the PCB
Parts:
- removed C1, C4: 100uF, ~, symbol C
- removed U1: MCP16321/2, ~, symbol MCP16321/2
- removed U3: 3.3V OUT, symbol WIRE2
- added C1, C4: 100uF, ~, symbol CP1
- added C5: 4.7uF, ~, symbol C
- added U1, U4: 12V OUT, symbol WIRE2
- added U3: MCP16321/2, ~, symbol MCP16321/2
- added U5: 3.3V OUT, symbol WIRE2
- C2: value 20uF -> 4.7uF
- U2: value 12V OUT -> 3.3V OUT
Connections:
- net 12V: now also C1.1, C5.1, U1.1, U3.2 (VIN), U4.1; no longer U2.1
- net 3.3V: now also U2.1, C4.1, U3.5 (FB), U5.1
- net GND: now also C1.2, C4.2, C5.2, U1.2, U3.15 (PGND), U3.17 (EP), U3.4 (SGND), U4.2, U5.2
- net at C3.1: now also U3.10 (BOOST)
- net at L1.2: now also U3.12 (SW)

Commit message: 8-25
Parts:
- F1: value 20A -> 7A
Changed lines of the file:
@@
 LIBS:CustomConnect
 LIBS:CustomPower
+LIBS:Scoreboard_PowerSupply-cache
 EELAYER 27 0
 EELAYER END
@@
 $EndComp
 $Comp
-L GND #PWR1
+L GND #PWR01
 U 1 1 53FA573F
 P 3400 3950
-F 0 "#PWR1" H 3400 3950 30  0001 C CNN
+F 0 "#PWR01" H 3400 3950 30  0001 C CNN
 F 1 "GND" H 3400 3880 30  0001 C CNN
 F 2 "" H 3400 3950 60  0000 C CNN
@@
 $EndComp
 $Comp
-L GND #PWR4
+L GND #PWR02
 U 1 1 53FA5741
 P 4450 4300
-F 0 "#PWR4" H 4450 4300 30  0001 C CNN
+F 0 "#PWR02" H 4450 4300 30  0001 C CNN
 F 1 "GND" H 4450 4230 30  0001 C CNN
 F 2 "" H 4450 4300 60  0000 C CNN
@@
 P 3750 3500
 F 0 "F1" H 3850 3550 40  0000 C CNN
-F 1 "20A" H 3650 3450 40  0000 C CNN
+F 1 "7A" H 3650 3450 40  0000 C CNN
 F 2 "~" H 3750 3500 60  0000 C CNN
 F 3 "~" H 3750 3500 60  0000 C CNN
@@
 $EndComp
 $Comp
-L GND #PWR3
+L GND #PWR03
 U 1 1 53FA5745
 P 4150 4300
-F 0 "#PWR3" H 4150 4300 30  0001 C CNN
+F 0 "#PWR03" H 4150 4300 30  0001 C CNN
 F 1 "GND" H 4150 4230 30  0001 C CNN
 F 2 "" H 4150 4300 60  0000 C CNN
@@
 $EndComp
 $Comp
-L GND #PWR8
+L GND #PWR04
 U 1 1 53FA5746
 P 6450 4500
-F 0 "#PWR8" H 6450 4500 30  0001 C CNN
+F 0 "#PWR04" H 6450 4500 30  0001 C CNN
 F 1 "GND" H 6450 4430 30  0001 C CNN
 F 2 "" H 6450 4500 60  0000 C CNN
@@
 $EndComp
 $Comp
-L GND #PWR9
+L GND #PWR05
 U 1 1 53FA5747
 P 6700 4500
-F 0 "#PWR9" H 6700 4500 30  0001 C CNN
+F 0 "#PWR05" H 6700 4500 30  0001 C CNN
 F 1 "GND" H 6700 4430 30  0001 C CNN
 F 2 "" H 6700 4500 60  0000 C CNN
@@
 3.3V
 $Comp
-L GND #PWR12
+L GND #PWR06
 U 1 1 53FA574B
 P 8300 4200
-F 0 "#PWR12" H 8300 4200 30  0001 C CNN
+F 0 "#PWR06" H 8300 4200 30  0001 C CNN
 F 1 "GND" H 8300 4130 30  0001 C CNN
 F 2 "" H 8300 4200 60  0000 C CNN
@@
 $EndComp
 $Comp
-L GND #PWR6
+L GND #PWR07
 U 1 1 53FA574D
 P 5400 4200
-F 0 "#PWR6" H 5400 4200 30  0001 C CNN
+F 0 "#PWR07" H 5400 4200 30  0001 C CNN
 F 1 "GND" H 5400 4130 30  0001 C CNN
 F 2 "" H 5400 4200 60  0000 C CNN
@@
 $EndComp
 $Comp
-L GND #PWR7
+L GND #PWR08
 U 1 1 53FA574E
 P 5850 4500
-F 0 "#PWR7" H 5850 4500 30  0001 C CNN
+F 0 "#PWR08" H 5850 4500 30  0001 C CNN
 F 1 "GND" H 5850 4430 30  0001 C CNN
 F 2 "" H 5850 4500 60  0000 C CNN
@@
 $EndComp
 $Comp
-L GND #PWR10
+L GND #PWR09
 U 1 1 53FA5751
 P 6800 5800
-F 0 "#PWR10" H 6800 5800 30  0001 C CNN
+F 0 "#PWR09" H 6800 5800 30  0001 C CNN
 F 1 "GND" H 6800 5730 30  0001 C CNN
 F 2 "" H 6800 5800 60  0000 C CNN
@@
 $EndComp
 $Comp
-L GND #PWR5
+L GND #PWR010
 U 1 1 53FA5752
 P 5100 5800
-F 0 "#PWR5" H 5100 5800 30  0001 C CNN
+F 0 "#PWR010" H 5100 5800 30  0001 C CNN
 F 1 "GND" H 5100 5730 30  0001 C CNN
 F 2 "" H 5100 5800 60  0000 C CNN
@@
 $EndComp
 $Comp
-L GND #PWR11
+L GND #PWR011
 U 1 1 53FA57FF
 P 8100 5850
-F 0 "#PWR11" H 8100 5850 30  0001 C CNN
+F 0 "#PWR011" H 8100 5850 30  0001 C CNN
 F 1 "GND" H 8100 5780 30  0001 C CNN
 F 2 "" H 8100 5850 60  0000 C CNN
@@
 $EndComp
 $Comp
-L GND #PWR2
+L GND #PWR012
 U 1 1 53FA580E
 P 3600 5800
-F 0 "#PWR2" H 3600 5800 30  0001 C CNN
+F 0 "#PWR012" H 3600 5800 30  0001 C CNN
 F 1 "GND" H 3600 5730 30  0001 C CNN
 F 2 "" H 3600 5800 60  0000 C CNN

Commit message: 8-25 10:02
Connections:
- net at L1.2, U3.12 (SW): now also C3.2
Changed lines of the file:
@@
 LIBS:CustomConnect
 LIBS:CustomPower
+LIBS:WF121
 LIBS:Scoreboard_PowerSupply-cache
 EELAYER 27 0
@@
 Sheet 1 1
 Title ""
-Date "24 aug 2014"
+Date "26 aug 2014"
 Rev ""
 Comp ""
@@
 	0    1    1    0
 $EndComp
-Text HLabel 8750 3550 2    39   Input ~ 0
-3.3V
 $Comp
 L GND #PWR06
@@
 	1    0    0    -1
 $EndComp
-Text HLabel 6800 5350 0    39   Output ~ 0
-3.3V
-Text HLabel 5150 5350 0    39   Output ~ 0
-12V
-Text HLabel 4750 3100 1    39   Input ~ 0
-12V
 Wire Wire Line
 	3200 3700 3400 3700
@@
 Wire Wire Line
 	5100 5650 5100 5800
-Wire Wire Line
-	6950 5350 6800 5350
 Wire Wire Line
 	5300 5350 5150 5350
@@
 	1    0    0    -1
 $EndComp
-Text HLabel 3550 5350 0    39   Output ~ 0
-12V
-Text HLabel 8000 5350 0    39   Output ~ 0
-3.3V
 Wire Wire Line
 	8250 5350 8000 5350
-Wire Wire Line
-	3850 5350 3550 5350
 Wire Wire Line
 	3850 5650 3600 5650
@@
 Wire Wire Line
 	5150 4050 5400 4050
+Wire Wire Line
+	6800 5350 6950 5350
+Wire Wire Line
+	3850 5350 3550 5350
+Text GLabel 3550 5350 0    39   Output ~ 0
+12V
+Text GLabel 4750 3100 1    39   Output ~ 0
+12V
+Text GLabel 5150 5350 0    39   Output ~ 0
+12V
+Text GLabel 6800 5350 0    39   Output ~ 0
+3.3V
+Text GLabel 8000 5350 0    39   Output ~ 0
+3.3V
+Text GLabel 8750 3550 2    39   Input ~ 0
+3.3V
+Connection ~ 7050 3550
 $EndSCHEMATC
