File: PowerSupply/Scoreboard_PowerSupply.kicad_pcb (KiCad board)
At the start: 2 copper layers, 14 parts, among them CON1 12V INPUT, U1 12V OUT, U2 3.3V OUT, U3 MCP16321/2, U4 12V OUT, U5 3.3V OUT

Commit message: 8-25 10:02
Parts:
- added 1PIN: P***, 1pin, F.Cu at (237.4, 62.5)
- added 1PIN: P***, 1pin, F.Cu at (195.9, 75.0)
- moved C3 13.0 mm to (228.1, 66.2), turned to 90 degrees
- moved L1 9.43 mm to (234.3, 77.1), turned to 45 degrees
- moved C1 8.58 mm to (219.0, 71.2)
- moved C4 8.30 mm to (228.0, 64.1), turned to 270 degrees
- moved C2 7.92 mm to (216.5, 67.1), turned to 270 degrees
- moved D1 7.08 mm to (202.4, 80.9)
- moved U3 6.20 mm to (224.5, 69.0)
- moved C5 4.80 mm to (219.3, 67.1), turned to 270 degrees
- moved U2 3.70 mm to (238.1, 87.0)
- moved U5 3.56 mm to (238.1, 80.3)
- moved CON1 1.09 mm to (198.3, 64.8)
Connections:
- C1 pad 1: /12V -> 12V
- C2 pad 1: /12V -> 12V
- C3 pad 2: (no net) -> N-000004
- C4 pad 1: /3.3V -> 3.3V
- C5 pad 1: /12V -> 12V
- D1 pad 2: /12V -> 12V
- F1 pad 2: /12V -> 12V
- L1 pad 1: /3.3V -> 3.3V
- U1 pad 1: (no net) -> 12V
- U2 pad 1: (no net) -> 3.3V
- U3 pad 2: /12V -> 12V
- U3 pad 5: /3.3V -> 3.3V
- U4 pad 1: (no net) -> 12V
- U5 pad 1: (no net) -> 3.3V
Routing:
- net 12V: track 0.00 -> 56.0 mm
- net 3.3V: track 0.00 -> 35.1 mm
- net /12V: track 16.6 -> 0.00 mm
- net GND: track 0.00 -> 15.3 mm
- net N-000004: track 0.00 -> 13.9 mm
- net N-000003: track 0.00 -> 3.84 mm
- net N-000006: track 6.98 -> 7.82 mm
- added copper zone on B.Cu, net GND
- added copper zone on F.Cu, net GND
Other:
- board outline added: 49.1 x 19.3 mm
- net class 12V: clearance 0.254 -> 0.1
- net class 2: clearance 0.254 -> 0.1
- net class Default: clearance 0.254 -> 0.1
- rule trace_clearance: 0.254 -> 0.1

Commit message: 8-26-14
Parts:
- moved D1 21.6 mm to (221.0, 70.0), turned to 180 degrees
- moved 1PIN 13.1 mm to (209.0, 74.6)
- moved C1 10.7 mm to (208.4, 72.7), turned to 0 degrees
- moved CON1 5.80 mm to (194.5, 69.1)
- moved F1 3.88 mm to (209.7, 66.5), turned to 0 degrees
Routing:
- net GND: track 15.3 -> 0.28 mm, vias 0 -> 9
- net 12V: track 56.0 -> 45.8 mm
- net N-000006: track 7.82 -> 13.0 mm
Other:
- board text added: "KRATZ INDUSTRIES - 3.3V SUPPLY - 8-25-14"
