File: LED Drive/High Side Drive.sch (KiCad schematic (older format))
At the start: 23 parts, among them P10 CONN_8, P9 CONN_8, Q33 NPN, U6 74HC595, U7 74HC595

Commit message: 9-4
Parts:
- added Q? (x15): NPN, ~, symbol NPN
- added Q? (x15): MOS_P, ~, symbol MOS_P
- added R? (x15): 10K, ~, symbol R
Connections:
- net labels removed: SINK1
- wire segments 75 -> 220

Commit message: 9-4
Changing the LED drive to Opto-coupled
Parts:
- R33, R34, R37, R38, R39, R40, R41: value 1K -> 10K
Connections:
- net SOURCE1: no longer Q?.D, Q?.D, Q?.D, Q?.D, Q?.D, Q?.D, Q?.D, Q?.D
- net SOURCE10: now also Q?.D
- net SOURCE11: now also Q?.D
- net SOURCE12: now also Q?.D
- net SOURCE13: now also Q?.D
- net SOURCE14: now also Q?.D
- net SOURCE15: now also Q?.D
- net SOURCE16: now also Q?.D
- net SOURCE9: now also Q?.D
Changed lines of the file:
@@
 $Descr A4 8268 11693 portrait
 encoding utf-8
-Sheet 2 3
+Sheet 2 4
 Title ""
-Date "4 sep 2014"
+Date "5 sep 2014"
 Rev ""
 Comp ""
@@
 P 3800 1700
 F 0 "R34" V 3880 1700 40  0000 C CNN
-F 1 "1K" V 3807 1701 40  0000 C CNN
+F 1 "10K" V 3807 1701 40  0000 C CNN
 F 2 "~" V 3730 1700 30  0000 C CNN
 F 3 "~" H 3800 1700 30  0000 C CNN
@@
 P 3800 1200
 F 0 "R33" V 3880 1200 40  0000 C CNN
-F 1 "1K" V 3807 1201 40  0000 C CNN
+F 1 "10K" V 3807 1201 40  0000 C CNN
 F 2 "~" V 3730 1200 30  0000 C CNN
 F 3 "~" H 3800 1200 30  0000 C CNN
@@
 P 3850 2300
 F 0 "R37" V 3930 2300 40  0000 C CNN
-F 1 "1K" V 3857 2301 40  0000 C CNN
+F 1 "10K" V 3857 2301 40  0000 C CNN
 F 2 "~" V 3780 2300 30  0000 C CNN
 F 3 "~" H 3850 2300 30  0000 C CNN
@@
 P 3850 2800
 F 0 "R38" V 3930 2800 40  0000 C CNN
-F 1 "1K" V 3857 2801 40  0000 C CNN
+F 1 "10K" V 3857 2801 40  0000 C CNN
 F 2 "~" V 3780 2800 30  0000 C CNN
 F 3 "~" H 3850 2800 30  0000 C CNN
@@
 P 3850 3400
 F 0 "R39" V 3930 3400 40  0000 C CNN
-F 1 "1K" V 3857 3401 40  0000 C CNN
+F 1 "10K" V 3857 3401 40  0000 C CNN
 F 2 "~" V 3780 3400 30  0000 C CNN
 F 3 "~" H 3850 3400 30  0000 C CNN
@@
 P 3850 3900
 F 0 "R40" V 3930 3900 40  0000 C CNN
-F 1 "1K" V 3857 3901 40  0000 C CNN
+F 1 "10K" V 3857 3901 40  0000 C CNN
 F 2 "~" V 3780 3900 30  0000 C CNN
 F 3 "~" H 3850 3900 30  0000 C CNN
@@
 P 3850 4500
 F 0 "R41" V 3930 4500 40  0000 C CNN
-F 1 "1K" V 3857 4501 40  0000 C CNN
+F 1 "10K" V 3857 4501 40  0000 C CNN
 F 2 "~" V 3780 4500 30  0000 C CNN
 F 3 "~" H 3850 4500 30  0000 C CNN
@@
 12V
 Text GLabel 5650 6200 2    39   Input ~ 0
-SOURCE1
+SOURCE9
 Wire Wire Line
 	5350 6200 5650 6200
@@
 12V
 Text GLabel 7200 6700 2    39   Input ~ 0
-SOURCE1
+SOURCE10
 Wire Wire Line
 	6900 6700 7200 6700
@@
 12V
 Text GLabel 5700 7300 2    39   Input ~ 0
-SOURCE1
+SOURCE11
 Wire Wire Line
 	5400 7300 5700 7300
@@
 12V
 Text GLabel 7200 7800 2    39   Input ~ 0
-SOURCE1
+SOURCE12
 Wire Wire Line
 	6900 7800 7200 7800
@@
 12V
 Text GLabel 5700 8400 2    39   Input ~ 0
-SOURCE1
+SOURCE13
 Wire Wire Line
 	5400 8400 5700 8400
@@
 12V
 Text GLabel 7200 8900 2    39   Input ~ 0
-SOURCE1
+SOURCE14
 Wire Wire Line
 	6900 8900 7200 8900
@@
 12V
 Text GLabel 5700 9500 2    39   Input ~ 0
-SOURCE1
+SOURCE15
 Wire Wire Line
 	5400 9500 5700 9500
@@
 Text GLabel 7250 9550 2    39   Input ~ 0
 12V
+Wire Wire Line
+	6900 10000 7200 10000
 Text GLabel 7200 10000 2    39   Input ~ 0
-SOURCE1
-Wire Wire Line
-	6900 10000 7200 10000
+SOURCE16
 $EndSCHEMATC
