File: LED Drive/HighSideIsolatedDrive.sch (KiCad schematic (older format))
At the start: 54 parts, among them Q1 MOS_N, Q10 MOS_N, Q11 MOS_N, Q12 MOS_N, Q13 MOS_N, Q14 MOS_N, Q15 MOS_N, Q16 MOS_N, Q2 MOS_N, Q3 MOS_N, Q4 MOS_N, Q5 MOS_N, Q6 MOS_N, Q7 MOS_N, Q8 MOS_N, Q9 MOS_N, U10 74LS595, U11 LTV847, U12 LTV847, U13 LTV847, U14 LTV847, U9 74LS595

Commit message: 9-8
Parts:
- removed Q1, Q10, Q11, Q12, Q13, Q14, Q15, Q16, Q2, Q3, Q4, Q5, Q6, Q7, Q8, Q9: MOS_N, ~, symbol MOS_N
- removed R1, R10, R11, R12, R13, R14, R15, R16, R2, R3, R4, R5, R6, R7, R8, R9: 330, ~, symbol R
- removed R17, R18, R19, R20, R21, R22, R23, R24, R25, R26, R27, R28, R29, R30, R31, R32: 10K, ~, symbol R
- removed U10, U9: 74LS595, ~, symbol 74LS595
- removed U11, U12, U13, U14: LTV847, symbol LTV847
- added Q17, Q18, Q19, Q20, Q21, Q22, Q23, Q24, Q25, Q26, Q27, Q28, Q29, Q30, Q31, Q32: MOS_P, ~, symbol MOS_P
- added R33, R34, R35, R36, R37, R38, R39, R40, R41, R42, R43, R44, R45, R46, R47, R48: 330, ~, symbol R
- added R49, R50, R51, R52, R53, R54, R55, R56, R57, R58, R59, R60, R61, R62, R63, R64: 10K, ~, symbol R
- added U15, U16: 74LS595, ~, symbol 74LS595
- added U17, U18, U19, U20: LTV847, symbol LTV847
Connections:
- net 12V: now also Q17.D, Q18.D, Q19.D, Q20.D, Q21.D, Q22.D, Q23.D, Q24.D, Q25.D, Q26.D, Q27.D, Q28.D, Q29.D, Q30.D, Q31.D, Q32.D, R49.1, R50.1, R51.1, R52.1, R53.1, R54.1, R55.1, R56.1, R57.1, R58.1, R59.1, R60.1, R61.1, R62.1, R63.1, R64.1
- net CLK: now also U15.11 (SRCLK), U16.11 (SRCLK)
- net GND: now also U15.13 (G), U16.13 (G), U17.11 (E), U17.13 (E), U17.15 (E), U17.2 (K), U17.4 (K), U17.6 (K), U17.8 (K), U17.9 (E), U18.11 (E), U18.13 (E), U18.15 (E), U18.2 (K), U18.4 (K), U18.6 (K), U18.8 (K), U18.9 (E), U19.11 (E), U19.13 (E), U19.15 (E), U19.2 (K), U19.4 (K), U19.6 (K), U19.8 (K), U19.9 (E), U20.11 (E), U20.13 (E), U20.15 (E), U20.2 (K), U20.4 (K), U20.6 (K), U20.8 (K), U20.9 (E)
- net STROBE: now also U15.12 (RCLK), U16.12 (RCLK)
- net VCC3.3: now also U15.10 (SRCLR), U16.10 (SRCLR)
- new net: R41.1, U17.1 (A)
- new net: Q26.G, R52.2, U17.10 (C)
- new net: Q18.G, R51.2, U17.12 (C)
- new net: Q25.G, R50.2, U17.14 (C)
- new net: Q17.G, R49.2, U17.16 (C)
- new net: R42.1, U17.3 (A)
- new net: R43.1, U17.5 (A)
- new net: R44.1, U17.7 (A)
- new net: R43.2, U15.2 (QC)
- new net: Q27.G, R54.2, U18.14 (C)
- new net: Q28.G, R56.2, U18.10 (C)
- new net: Q22.G, R59.2, U19.12 (C)
- new net: R37.1, U20.1 (A)
- new net: Q32.G, R64.2, U20.10 (C)
- new net: Q24.G, R63.2, U20.12 (C)
- new net: Q31.G, R62.2, U20.14 (C)
- new net: Q23.G, R61.2, U20.16 (C)
- new net: R38.1, U20.3 (A)
- new net: R39.1, U20.5 (A)
- new net: R40.1, U20.7 (A)
- new net: R37.2, U16.4 (QE)
- new net: R38.2, U16.5 (QF)
- new net: R39.2, U16.6 (QG)
- new net: R40.2, U16.7 (QH)
- new net: Q19.G, R53.2, U18.16 (C)
- new net: Q20.G, R55.2, U18.12 (C)
- new net: Q21.G, R57.2, U19.16 (C)
- new net: Q29.G, R58.2, U19.14 (C)
- new net: Q30.G, R60.2, U19.10 (C)
- new net: R42.2, U15.1 (QB)
- new net: R41.2, U15.15 (QA)
- new net: R44.2, U15.3 (QD)
- new net: R45.2, U15.4 (QE)
- new net: R46.2, U15.5 (QF)
- new net: R47.2, U15.6 (QG)
- new net: R48.2, U15.7 (QH)
- new net: U15.9 (~QH), U16.14 (SER)
- new net: R34.2, U16.1 (QB)
- new net: R33.2, U16.15 (QA)
- new net: R35.2, U16.2 (QC)
- new net: R36.2, U16.3 (QD)
- new net: R45.1, U18.1 (A)
- new net: R46.1, U18.3 (A)
- new net: R47.1, U18.5 (A)
- new net: R48.1, U18.7 (A)
- new net: R33.1, U19.1 (A)
- new net: R34.1, U19.3 (A)
- new net: R35.1, U19.5 (A)
- new net: R36.1, U19.7 (A)
- new net HS_IN: U15.14 (SER)
- new net HS_OUT: U16.9 (~QH)
- new net SOURCE1: Q17.S
- new net SOURCE10: Q29.S
- new net SOURCE11: Q22.S
- new net SOURCE12: Q30.S
- new net SOURCE13: Q23.S
- new net SOURCE14: Q31.S
- new net SOURCE15: Q24.S
- new net SOURCE16: Q32.S
- new net SOURCE2: Q25.S
- new net SOURCE3: Q18.S
- new net SOURCE4: Q26.S
- new net SOURCE5: Q19.S
- new net SOURCE6: Q20.S, Q27.S
- new net SOURCE8: Q28.S
- new net SOURCE9: Q21.S

Commit message: 9-16
Connections:
- net GND: now also U15.8 (GND), U16.8 (GND); no longer U17.11 (E), U17.13 (E), U17.15 (E), U17.9 (E), U18.11 (E), U18.13 (E), U18.15 (E), U18.9 (E), U19.11 (E), U19.13 (E), U19.15 (E), U19.9 (E), U20.11 (E), U20.13 (E), U20.15 (E), U20.9 (E)
- net SOURCE6: no longer Q20.S
- net VCC3.3: now also U15.16 (VCC), U16.16 (VCC)
- new net GND2: U17.11 (E), U17.13 (E), U17.15 (E), U17.9 (E), U18.11 (E), U18.13 (E), U18.15 (E), U18.9 (E), U19.11 (E), U19.13 (E), U19.15 (E), U19.9 (E), U20.11 (E), U20.13 (E), U20.15 (E), U20.9 (E)
- new net SOURCE7: Q20.S

Commit message: Finallizing LED Driver
Parts:
- added C3, C4: C, ~, symbol C
Connections:
- net GND: now also C3.2, C4.2
- net VCC3.3: now also C3.1, C4.1
Changed lines of the file:
@@
 Sheet 3 3
 Title ""
-Date "10 sep 2014"
+Date "26 sep 2014"
 Rev ""
 Comp ""
@@
 $EndComp
 $Comp
-L GND #PWR020
+L GND #PWR022
 U 1 1 540E5EB0
 P 1700 2300
-F 0 "#PWR020" H 1700 2300 30  0001 C CNN
+F 0 "#PWR022" H 1700 2300 30  0001 C CNN
 F 1 "GND" H 1700 2230 30  0001 C CNN
 F 2 "" H 1700 2300 60  0000 C CNN
@@
 $EndComp
 $Comp
-L GND #PWR021
+L GND #PWR023
 U 1 1 540E5EB1
 P 1700 4150
-F 0 "#PWR021" H 1700 4150 30  0001 C CNN
+F 0 "#PWR023" H 1700 4150 30  0001 C CNN
 F 1 "GND" H 1700 4080 30  0001 C CNN
 F 2 "" H 1700 4150 60  0000 C CNN
@@
 $EndComp
 $Comp
-L GND #PWR022
+L GND #PWR024
 U 1 1 540E5EB6
 P 4400 1350
-F 0 "#PWR022" H 4400 1350 30  0001 C CNN
+F 0 "#PWR024" H 4400 1350 30  0001 C CNN
 F 1 "GND" H 4400 1280 30  0001 C CNN
 F 2 "" H 4400 1350 60  0000 C CNN
@@
 $EndComp
 $Comp
-L GND #PWR023
+L GND #PWR025
 U 1 1 5409301B
 P 4400 1750
-F 0 "#PWR023" H 4400 1750 30  0001 C CNN
+F 0 "#PWR025" H 4400 1750 30  0001 C CNN
 F 1 "GND" H 4400 1680 30  0001 C CNN
 F 2 "" H 4400 1750 60  0000 C CNN
@@
 $EndComp
 $Comp
-L GND #PWR024
+L GND #PWR026
 U 1 1 5409302A
 P 4400 2150
-F 0 "#PWR024" H 4400 2150 30  0001 C CNN
+F 0 "#PWR026" H 4400 2150 30  0001 C CNN
 F 1 "GND" H 4400 2080 30  0001 C CNN
 F 2 "" H 4400 2150 60  0000 C CNN
@@
 $EndComp
 $Comp
-L GND #PWR025
+L GND #PWR027
 U 1 1 54093039
 P 4400 2500
-F 0 "#PWR025" H 4400 2500 30  0001 C CNN
+F 0 "#PWR027" H 4400 2500 30  0001 C CNN
 F 1 "GND" H 4400 2430 30  0001 C CNN
 F 2 "" H 4400 2500 60  0000 C CNN
@@
 $EndComp
 $Comp
-L GND #PWR026
+L GND #PWR028
 U 1 1 540E5EC7
 P 4400 3200
-F 0 "#PWR026" H 4400 3200 30  0001 C CNN
+F 0 "#PWR028" H 4400 3200 30  0001 C CNN
 F 1 "GND" H 4400 3130 30  0001 C CNN
 F 2 "" H 4400 3200 60  0000 C CNN
@@
 $EndComp
 $Comp
-L GND #PWR027
+L GND #PWR029
 U 1 1 540E5EC8
 P 4400 3600
-F 0 "#PWR027" H 4400 3600 30  0001 C CNN
+F 0 "#PWR029" H 4400 3600 30  0001 C CNN
 F 1 "GND" H 4400 3530 30  0001 C CNN
 F 2 "" H 4400 3600 60  0000 C CNN
@@
 $EndComp
 $Comp
-L GND #PWR028
+L GND #PWR030
 U 1 1 54093713
 P 4400 4000
-F 0 "#PWR028" H 4400 4000 30  0001 C CNN
+F 0 "#PWR030" H 4400 4000 30  0001 C CNN
 F 1 "GND" H 4400 3930 30  0001 C CNN
 F 2 "" H 4400 4000 60  0000 C CNN
@@
 $EndComp
 $Comp
-L GND #PWR029
+L GND #PWR031
 U 1 1 540E5ECA
 P 4400 4350
-F 0 "#PWR029" H 4400 4350 30  0001 C CNN
+F 0 "#PWR031" H 4400 4350 30  0001 C CNN
 F 1 "GND" H 4400 4280 30  0001 C CNN
 F 2 "" H 4400 4350 60  0000 C CNN
@@
 $EndComp
 $Comp
-L GND #PWR030
+L GND #PWR032
 U 1 1 540E5ED8
 P 4400 5150
-F 0 "#PWR030" H 4400 5150 30  0001 C CNN
+F 0 "#PWR032" H 4400 5150 30  0001 C CNN
 F 1 "GND" H 4400 5080 30  0001 C CNN
 F 2 "" H 4400 5150 60  0000 C CNN
@@
 $EndComp
 $Comp
-L GND #PWR031
+L GND #PWR033
 U 1 1 540E5ED9
 P 4400 5550
-F 0 "#PWR031" H 4400 5550 30  0001 C CNN
+F 0 "#PWR033" H 4400 5550 30  0001 C CNN
 F 1 "GND" H 4400 5480 30  0001 C CNN
 F 2 "" H 4400 5550 60  0000 C CNN
@@
 $EndComp
 $Comp
-L GND #PWR032
+L GND #PWR034
 U 1 1 540E5EDA
 P 4400 5950
-F 0 "#PWR032" H 4400 5950 30  0001 C CNN
+F 0 "#PWR034" H 4400 5950 30  0001 C CNN
 F 1 "GND" H 4400 5880 30  0001 C CNN
 F 2 "" H 4400 5950 60  0000 C CNN
@@
 $EndComp
 $Comp
-L GND #PWR033
+L GND #PWR035
 U 1 1 540E5EDB
 P 4400 6300
-F 0 "#PWR033" H 4400 6300 30  0001 C CNN
+F 0 "#PWR035" H 4400 6300 30  0001 C CNN
 F 1 "GND" H 4400 6230 30  0001 C CNN
 F 2 "" H 4400 6300 60  0000 C CNN
@@
 $EndComp
 $Comp
-L GND #PWR034
+L GND #PWR036
 U 1 1 540938A3
 P 4400 7000
-F 0 "#PWR034" H 4400 7000 30  0001 C CNN
+F 0 "#PWR036" H 4400 7000 30  0001 C CNN
 F 1 "GND" H 4400 6930 30  0001 C CNN
 F 2 "" H 4400 7000 60  0000 C CNN
@@
 $EndComp
 $Comp
-L GND #PWR035
+L GND #PWR037
 U 1 1 540938A9
 P 4400 7400
-F 0 "#PWR035" H 4400 7400 30  0001 C CNN
+F 0 "#PWR037" H 4400 7400 30  0001 C CNN
 F 1 "GND" H 4400 7330 30  0001 C CNN
 F 2 "" H 4400 7400 60  0000 C CNN
@@
 $EndComp
 $Comp
-L GND #PWR036
+L GND #PWR038
 U 1 1 540938AF
 P 4400 7800
-F 0 "#PWR036" H 4400 7800 30  0001 C CNN
+F 0 "#PWR038" H 4400 7800 30  0001 C CNN
 F 1 "GND" H 4400 7730 30  0001 C CNN
 F 2 "" H 4400 7800 60  0000 C CNN
@@
 $EndComp
 $Comp
-L GND #PWR037
+L GND #PWR039
 U 1 1 540938B5
 P 4400 8150
-F 0 "#PWR037" H 4400 8150 30  0001 C CNN
+F 0 "#PWR039" H 4400 8150 30  0001 C CNN
 F 1 "GND" H 4400 8080 30  0001 C CNN
 F 2 "" H 4400 8150 60  0000 C CNN
@@
 	2100 1000 2100 800
 Wire Wire Line
-	2100 800  1250 800
+	1250 800  2200 800
 Connection ~ 1250 1400
 Wire Wire Line
-	2100 2800 2100 2650
+	2100 2600 2100 2800
 Wire Wire Line
 	2100 2650 1250 2650
@@
 	2100 4000 1700 4000
 Connection ~ 1700 4000
+$Comp
+L C C3
+U 1 1 5424D902
+P 2400 800
+F 0 "C3" H 2400 900 40  0000 L CNN
+F 1 "C" H 2406 715 40  0000 L CNN
+F 2 "~" H 2438 650 30  0000 C CNN
+F 3 "~" H 2400 800 60  0000 C CNN
+	1    2400 800
+	0    -1   -1   0
+$EndComp
+$Comp
+L GND #PWR040
+U 1 1 5424D911
+P 2700 800
+F 0 "#PWR040" H 2700 800 30  0001 C CNN
+F 1 "GND" H 2700 730 30  0001 C CNN
+F 2 "" H 2700 800 60  0000 C CNN
+F 3 "" H 2700 800 60  0000 C CNN
+	1    2700 800
+	0    -1   -1   0
+$EndComp
+Connection ~ 2100 800
+Wire Wire Line
+	2600 800  2700 800
+$Comp
+L C C4
+U 1 1 5424DB53
+P 2350 2600
+F 0 "C4" H 2350 2700 40  0000 L CNN
+F 1 "C" H 2356 2515 40  0000 L CNN
+F 2 "~" H 2388 2450 30  0000 C CNN
+F 3 "~" H 2350 2600 60  0000 C CNN
+	1    2350 2600
+	0    -1   -1   0
+$EndComp
+$Comp
+L GND #PWR041
+U 1 1 5424DB62
+P 2650 2600
+F 0 "#PWR041" H 2650 2600 30  0001 C CNN
+F 1 "GND" H 2650 2530 30  0001 C CNN
+F 2 "" H 2650 2600 60  0000 C CNN
+F 3 "" H 2650 2600 60  0000 C CNN
+	1    2650 2600
+	0    -1   -1   0
+$EndComp
+Wire Wire Line
+	2150 2600 2100 2600
+Connection ~ 2100 2650
+Wire Wire Line
+	2550 2600 2650 2600
 $EndSCHEMATC
