File: LED Drive/LowSideIsolatedDrive.sch (KiCad schematic (older format))
At the start: 54 parts, among them Q1 MOS_N, Q10 MOS_N, Q11 MOS_N, Q12 MOS_N, Q13 MOS_N, Q14 MOS_N, Q15 MOS_N, Q16 MOS_N, Q2 MOS_N, Q3 MOS_N, Q4 MOS_N, Q5 MOS_N, Q6 MOS_N, Q7 MOS_N, Q8 MOS_N, Q9 MOS_N, U10 74LS595, U11 LTV847, U12 LTV847, U13 LTV847, U14 LTV847, U9 74LS595

Commit message: 9-16
Connections:
- net GND: now also U10.8 (GND), U9.8 (GND); no longer Q1.S, Q10.S, Q11.S, Q12.S, Q13.S, Q14.S, Q15.S, Q16.S, Q2.S, Q3.S, Q4.S, Q5.S, Q6.S, Q7.S, Q8.S, Q9.S, U11.11 (E), U11.13 (E), U11.15 (E), U11.9 (E), U12.11 (E), U12.13 (E), U12.15 (E), U12.9 (E), U13.11 (E), U13.13 (E), U13.15 (E), U13.9 (E), U14.11 (E), U14.13 (E), U14.15 (E), U14.9 (E)
- net VCC3.3: now also U10.16 (VCC), U9.16 (VCC)
- new net GND2: Q1.S, Q10.S, Q11.S, Q12.S, Q13.S, Q14.S, Q15.S, Q16.S, Q2.S, Q3.S, Q4.S, Q5.S, Q6.S, Q7.S, Q8.S, Q9.S, U11.11 (E), U11.13 (E), U11.15 (E), U11.9 (E), U12.11 (E), U12.13 (E), U12.15 (E), U12.9 (E), U13.11 (E), U13.13 (E), U13.15 (E), U13.9 (E), U14.11 (E), U14.13 (E), U14.15 (E), U14.9 (E)

Commit message: Finallizing LED Driver
Parts:
- added C1, C2: C, ~, symbol C
Connections:
- net GND: now also C1.1, C2.1
- net VCC3.3: now also C1.2, C2.2
Changed lines of the file:
@@
 Sheet 2 3
 Title ""
-Date "10 sep 2014"
+Date "26 sep 2014"
 Rev ""
 Comp ""
@@
 	7300 7900 7300 8000
 Wire Wire Line
-	2100 1000 2100 900
+	2100 750  2100 1000
 Wire Wire Line
 	2100 900  1250 900
@@
 	2100 2800 2100 2600
 Wire Wire Line
-	2100 2600 1250 2600
+	1250 2600 2150 2600
 Connection ~ 1250 2600
 Wire Wire Line
@@
 	2100 2200 1700 2200
 Connection ~ 1700 2200
+$Comp
+L C C1
+U 1 1 5424D432
+P 2300 750
+F 0 "C1" H 2300 850 40  0000 L CNN
+F 1 "C" H 2306 665 40  0000 L CNN
+F 2 "~" H 2338 600 30  0000 C CNN
+F 3 "~" H 2300 750 60  0000 C CNN
+	1    2300 750
+	0    1    1    0
+$EndComp
+$Comp
+L GND #PWR020
+U 1 1 5424D450
+P 2650 750
+F 0 "#PWR020" H 2650 750 30  0001 C CNN
+F 1 "GND" H 2650 680 30  0001 C CNN
+F 2 "" H 2650 750 60  0000 C CNN
+F 3 "" H 2650 750 60  0000 C CNN
+	1    2650 750
+	1    0    0    -1
+$EndComp
+Connection ~ 2100 900
+Wire Wire Line
+	2500 750  2650 750
+$Comp
+L C C2
+U 1 1 5424D698
+P 2350 2600
+F 0 "C2" H 2350 2700 40  0000 L CNN
+F 1 "C" H 2356 2515 40  0000 L CNN
+F 2 "~" H 2388 2450 30  0000 C CNN
+F 3 "~" H 2350 2600 60  0000 C CNN
+	1    2350 2600
+	0    1    1    0
+$EndComp
+$Comp
+L GND #PWR021
+U 1 1 5424D6B6
+P 2650 2600
+F 0 "#PWR021" H 2650 2600 30  0001 C CNN
+F 1 "GND" H 2650 2530 30  0001 C CNN
+F 2 "" H 2650 2600 60  0000 C CNN
+F 3 "" H 2650 2600 60  0000 C CNN
+	1    2650 2600
+	0    -1   1    0
+$EndComp
+Connection ~ 2100 2600
+Wire Wire Line
+	2550 2600 2650 2600
 $EndSCHEMATC
