File: LED Drive/LED Drive.kicad_pcb (KiCad board)
At the start: 2 copper layers, 116 parts, among them Q1 MOS_N, Q10 MOS_N, Q11 MOS_N, Q12 MOS_N, Q13 MOS_N, Q14 MOS_N, Q15 MOS_N, Q16 MOS_N, Q17 MOS_P, Q18 MOS_P, Q19 MOS_P, Q2 MOS_N, Q20 MOS_P, Q21 MOS_P, Q22 MOS_P, Q23 MOS_P, Q24 MOS_P, Q25 MOS_P, Q26 MOS_P, Q27 MOS_P, Q28 MOS_P, Q29 MOS_P, Q3 MOS_N, Q30 MOS_P, Q31 MOS_P, Q32 MOS_P, Q4 MOS_N, Q5 MOS_N, Q6 MOS_N, Q7 MOS_N, Q8 MOS_N, Q9 MOS_N, U1 LOW_1-8, U10 74LS595, U11 LTV847, U12 LTV847, U13 LTV847, U14 LTV847, U15 74LS595, U16 74LS595, U17 LTV847, U18 LTV847, U19 LTV847, U2 LOW_9-16, U20 LTV847, U3 HIGH_1-8, U4 HIGH_9-16, U5 DATA, U6 3.3V, U7 12V, U8 DATA_OUT, U9 74LS595

Commit message: Finallizing LED Driver
Parts:
- added C1: C, SM0603_Capa, F.Cu at (191.0, 54.1)
- added C2: C, SM0603_Capa, F.Cu at (190.0, 104.8)
- added C3: C, SM0603_Capa, F.Cu at (191.0, 151.6)
- added C4: C, SM0603_Capa, F.Cu at (191.0, 200.2)
- U10, U15, U16, U9: moved to B.Cu
- moved U7 132.9 mm to (222.9, 29.2), turned to 90 degrees
- moved U16 117.9 mm to (192.3, 203.7)
- moved U15 108.9 mm to (192.0, 155.2), turned to 270 degrees
- moved U8 107.4 mm to (200.8, 227.6), turned to 90 degrees
- moved U10 43.1 mm to (192.0, 106.2), turned to 270 degrees
- moved U9 31.8 mm to (192.0, 57.4), turned to 270 degrees
- moved U5 17.8 mm to (184.3, 29.0)
- moved U6 14.5 mm to (202.1, 32.8)
Routing:
- net 12V: track 0.00 -> 448.9 mm, vias 0 -> 32
- net VCC3.3: track 8.07 -> 223.2 mm, vias 0 -> 8
- net CLK: track 15.5 -> 203.7 mm, vias 0 -> 3
- net STROBE: track 19.8 -> 187.4 mm
- net HS_IN: track 0.00 -> 132.5 mm, vias 0 -> 2
- net LS_OUT: track 0.00 -> 132.2 mm, vias 0 -> 1
- net N-0000087: track 0.00 -> 50.6 mm, vias 0 -> 2
- net N-00000131: track 0.00 -> 49.0 mm, vias 0 -> 2
- net N-0000075: track 52.4 -> 19.5 mm, vias 2 -> 1
- net N-0000074: track 47.2 -> 15.6 mm, vias 2 -> 1
- net N-0000073: track 41.3 -> 11.3 mm, vias 2 -> 1
- net N-0000072: track 35.5 -> 10.1 mm, vias 2 -> 1
- net N-00000126: track 0.00 -> 24.3 mm, vias 0 -> 1
- net HS_OUT: track 0.00 -> 24.2 mm
- net N-00000102: track 0.00 -> 23.8 mm, vias 0 -> 1
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- added copper zone on B.Cu, net GND
- added copper zone on F.Cu, net GND
- added copper zone on B.Cu, net GND2
- added copper zone on F.Cu, net GND2
Other:
- board outline added: 32 x 202.4 mm
- board text added: "KRATZ INDUSTRIES - ISOLATED POWER DRIVER ARRAY"

Commit message: Still finalizng LED Driver
Routing:
- net GND: track 0.13 -> 93.9 mm, vias 25 -> 28
- net GND2: track 0.00 -> 90.1 mm
- net (no net): track 0.13 -> 5.71 mm, vias 0 -> 2
- net LS_OUT: track 132.2 -> 133.6 mm
- net N-00000108: track 9.62 -> 10.2 mm

Commit message: 10-2-14
Parts:
- added HOLE: VAL**, HOLE, F.Cu at (215.9, 226.6)
- added HOLE: VAL**, HOLE, F.Cu at (216.4, 33.5)
- added HOLE: VAL**, HOLE, F.Cu at (188.5, 36.6)
- added HOLE: VAL**, HOLE, F.Cu at (188.3, 223.4)
- added HOLE: VAL**, HOLE, F.Cu at (206.4, 130.4)
- moved R9 1.63 mm to (192.3, 37.6), turned to 270 degrees
- moved R40 1.45 mm to (191.9, 223.6), turned to 90 degrees
Routing:
- net GND: track 93.9 -> 119.0 mm, vias 28 -> 34
- net (no net): track 5.71 -> 0.00 mm, vias 2 -> 0
- net N-00000126: track 24.3 -> 19.9 mm
- net GND2: track 90.1 -> 92.3 mm
- net VCC3.3: track 223.2 -> 224.7 mm
- net N-0000099: track 2.43 -> 3.37 mm

Commit message: Test Display Finished
Routing:
- net 12V: track 448.9 -> 451.0 mm
Changed lines of the file:
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@@
   (general
     (links 326)
-    (no_connects 1)
-    (area -3.106777 -1.524 229.567714 229.616001)
+    (no_connects 0)
+    (area 168.196286 25.4 229.567714 229.616001)
     (thickness 1.6)
     (drawings 5)
-    (tracks 1312)
+    (tracks 1314)
     (zones 0)
     (modules 125)
@@
   )
   (setup
-    (last_trace_width 0.254)
+    (last_trace_width 0.762)
     (user_trace_width 0.254)
     (user_trace_width 0.381)
@@
   (gr_line (start 186.563 229.108) (end 186.563 26.67) (angle 90) (layer Edge.Cuts) (width 0.1))
   (gr_line (start 218.567 26.67) (end 218.567 229.108) (angle 90) (layer Edge.Cuts) (width 0.1))
+  (segment (start 211.11464 214.884) (end 211.11464 213.01964) (width 0.762) (layer F.Cu) (net 1) (status 400000))
+  (segment (start 211.11464 213.01964) (end 210.947 212.852) (width 0.762) (layer F.Cu) (net 1))
   (segment (start 207.264 36.576) (end 207.264 34.544) (width 0.762) (layer F.Cu) (net 1))
   (segment (start 207.772 34.036) (end 210.185 34.036) (width 0.762) (layer B.Cu) (net 1))
