File: TestDisplay/TestDisplay.sch (KiCad schematic (older format))
At the start: 90 parts

Commit message: Test display
Parts:
- added C1: 10uF, ~, symbol C
- added C2, C3: 1uF, ~, symbol C
- added P1: CONN_6, symbol CONN_6
- added R15, R16, R17, R18, R19, R20, R21, R22, R58, R59, R60, R61, R62, R63, R64, R65: 1K, ~, symbol R
- added U2: 7805, ~, symbol 7805
- gave numbers to parts that had none: 90
Connections:
- net GND: now also U1.13 (G), U1.8 (GND), U3.13 (G), U3.8 (GND), C1.2, C2.2, C3.2, P1.1, U2.GND
- net VCC: now also C1.1, P1.2, U2.VI
- net at U1.1 (QB): now also R16.1; no longer Q3.2 (B)
- net V3.3: now reaches U1.10 (SRCLR)
- net V3.3: now also U1.16 (VCC), U3.10 (SRCLR), U3.16 (VCC), C2.1, C3.1, U2.VO
- net CLK: now reaches U1.11 (SRCLK)
- net CLK: now also U3.11 (SRCLK), P1.5
- net STROBE: now reaches U1.12 (RCLK)
- net STROBE: now also U3.12 (RCLK), P1.6
- net DATA1: now reaches U1.14 (SER)
- net DATA1: now also P1.3
- net at U1.15 (QA): now also R15.1; no longer Q1.2 (B)
- net at U1.2 (QC): now also R17.1; no longer Q5.2 (B)
- net at U1.3 (QD): now also R18.1; no longer Q7.2 (B)
- net at U1.4 (QE): now also R19.1; no longer Q8.2 (B)
- net at U1.5 (QF): now also R20.1; no longer Q6.2 (B)
- net at U1.6 (QG): now also R21.1; no longer Q4.2 (B)
- net at U1.7 (QH): now also R22.1; no longer Q2.2 (B)
- net at U3.1 (QB): now also R59.1; no longer Q11.2 (B)
- net DATA2: now reaches U3.14 (SER)
- net DATA2: now also P1.4
- net at U3.15 (QA): now also R58.1; no longer Q9.2 (B)
- net at U3.2 (QC): now also R60.1; no longer Q13.2 (B)
- net at U3.3 (QD): now also R61.1; no longer Q15.2 (B)
- net at U3.4 (QE): now also R62.1; no longer Q16.2 (B)
- net at U3.5 (QF): now also R63.1; no longer Q14.2 (B)
- net at U3.6 (QG): now also R64.1; no longer Q12.2 (B)
- net at U3.7 (QH): now also R65.1; no longer Q10.2 (B)
- new net: Q1.2 (B), R15.2
- new net: Q3.2 (B), R16.2
- new net: Q5.2 (B), R17.2
- new net: Q7.2 (B), R18.2
- new net: Q2.2 (B), R22.2
- new net: Q4.2 (B), R21.2
- new net: Q6.2 (B), R20.2
- new net: Q8.2 (B), R19.2
- new net: Q9.2 (B), R58.2
- new net: Q11.2 (B), R59.2
- new net: Q13.2 (B), R60.2
- new net: Q15.2 (B), R61.2
- new net: Q10.2 (B), R65.2
- new net: Q12.2 (B), R64.2
- new net: Q14.2 (B), R63.2
- new net: Q16.2 (B), R62.2
Other:
- moved on the sheet: AFF1, AFF2, AFF3, AFF4, AFF5, AFF6, AFF7, AFF8, AFF9, Q1, Q10, Q11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

Commit message: Daily
Parts:
- removed Q1, Q10, Q11, Q12, Q13, Q14, Q15, Q16, Q2, Q3, Q4, Q5, Q6, Q7, Q8, Q9: NPN, ~, symbol NPN
- added Q1, Q10, Q11, Q12, Q13, Q14, Q15, Q16, Q2, Q3, Q4, Q5, Q6, Q7, Q8, Q9: MMBT6427, ~, symbol MMBT6427
Connections:
- net 1: now also Q9.2 (E)
- net 2: now also Q11.2 (E)
- net 3: now also Q13.2 (E)
- net 4: now also Q15.2 (E)
- net 5: now also Q16.2 (E)
- net 6: now also Q14.2 (E)
- net 7: now also Q12.2 (E)
- net 8: now also Q10.2 (E)
- net 9: now also Q2.2 (E)
- net A: now also Q1.3 (C)
- net B: now also Q3.3 (C)
- net C: now also Q5.3 (C)
- net D: now also Q7.3 (C)
- net E: now also Q8.3 (C)
- net F: now also Q6.3 (C)
- net GND: now also Q1.2 (E), Q3.2 (E), Q4.2 (E), Q5.2 (E), Q6.2 (E), Q7.2 (E), Q8.2 (E)
- net H: now also Q4.3 (C)
- net VCC: now also Q10.3 (C), Q11.3 (C), Q12.3 (C), Q13.3 (C), Q14.3 (C), Q15.3 (C), Q16.3 (C), Q2.3 (C), Q9.3 (C)
- net at R15.2: now also Q1.1 (B)
- net at R16.2: now also Q3.1 (B)
- net at R17.2: now also Q5.1 (B)
- net at R18.2: now also Q7.1 (B)
- net at R22.2: now also Q2.1 (B)
- net at R21.2: now also Q4.1 (B)
- net at R20.2: now also Q6.1 (B)
- net at R19.2: now also Q8.1 (B)
- net at R58.2: now also Q9.1 (B)
- net at R59.2: now also Q11.1 (B)
- net at R60.2: now also Q13.1 (B)
- net at R61.2: now also Q15.1 (B)
- net at R65.2: now also Q10.1 (B)
- net at R64.2: now also Q12.1 (B)
- net at R63.2: now also Q14.1 (B)
- net at R62.2: now also Q16.1 (B)
Changed lines of the file:
@@
 LIBS:contrib
 LIBS:valves
+LIBS:Custom
+LIBS:TestDisplay-cache
 EELAYER 27 0
 EELAYER END
@@
 Sheet 1 1
 Title ""
-Date "26 jan 2015"
+Date "27 jan 2015"
 Rev ""
 Comp ""
@@
 $EndComp
 $Comp
-L NPN Q1
-U 1 1 54C47FCB
-P 5500 5750
-F 0 "Q1" H 5500 5600 50  0000 R CNN
-F 1 "NPN" H 5500 5900 50  0000 R CNN
-F 2 "~" H 5500 5750 60  0000 C CNN
-F 3 "~" H 5500 5750 60  0000 C CNN
-	1    5500 5750
-	0    -1   -1   0
-$EndComp
-$Comp
 L GND #PWR9
 U 1 1 54C4804B
@@
 $EndComp
 $Comp
-L NPN Q3
-U 1 1 54C4822D
-P 6050 5850
-F 0 "Q3" H 6050 5700 50  0000 R CNN
-F 1 "NPN" H 6050 6000 50  0000 R CNN
-F 2 "~" H 6050 5850 60  0000 C CNN
-F 3 "~" H 6050 5850 60  0000 C CNN
-	1    6050 5850
-	0    -1   -1   0
-$EndComp
-$Comp
 L GND #PWR11
 U 1 1 54C48233
@@
 $EndComp
 $Comp
-L NPN Q5
-U 1 1 54C4823A
-P 6600 5950
-F 0 "Q5" H 6600 5800 50  0000 R CNN
-F 1 "NPN" H 6600 6100 50  0000 R CNN
-F 2 "~" H 6600 5950 60  0000 C CNN
-F 3 "~" H 6600 5950 60  0000 C CNN
-	1    6600 5950
-	0    -1   -1   0
-$EndComp
-$Comp
 L GND #PWR13
 U 1 1 54C48240
@@
 $EndComp
 $Comp
-L NPN Q7
-U 1 1 54C48247
-P 7150 6050
-F 0 "Q7" H 7150 5900 50  0000 R CNN
-F 1 "NPN" H 7150 6200 50  0000 R CNN
-F 2 "~" H 7150 6050 60  0000 C CNN
-F 3 "~" H 7150 6050 60  0000 C CNN
-	1    7150 6050
-	0    -1   -1   0
-$EndComp
-$Comp
 L GND #PWR15
 U 1 1 54C4824D
@@
 	1    7400 5950
 	0    -1   -1   0
-$EndComp
-$Comp
-L NPN Q2
-U 1 1 54C48254
-P 5500 6850
-F 0 "Q2" H 5500 6700 50  0000 R CNN
-F 1 "NPN" H 5500 7000 50  0000 R CNN
-F 2 "~" H 5500 6850 60  0000 C CNN
-F 3 "~" H 5500 6850 60  0000 C CNN
-	1    5500 6850
-	0    -1   1    0
-$EndComp
-$Comp
-L NPN Q4
-U 1 1 54C48318
-P 6050 6750
-F 0 "Q4" H 6050 6600 50  0000 R CNN
-F 1 "NPN" H 6050 6900 50  0000 R CNN
-F 2 "~" H 6050 6750 60  0000 C CNN
-F 3 "~" H 6050 6750 60  0000 C CNN
-	1    6050 6750
-	0    1    1    0
 $EndComp
 $Comp
@@
 $EndComp
 $Comp
-L NPN Q6
-U 1 1 54C48325
-P 6600 6650
-F 0 "Q6" H 6600 6500 50  0000 R CNN
-F 1 "NPN" H 6600 6800 50  0000 R CNN
-F 2 "~" H 6600 6650 60  0000 C CNN
-F 3 "~" H 6600 6650 60  0000 C CNN
-	1    6600 6650
-	0    1    1    0
-$EndComp
-$Comp
 L GND #PWR12
 U 1 1 54C4832B
@@
 F 3 "" H 6350 6750 60  0000 C CNN
 	1    6350 6750
-	0    1    1    0
-$EndComp
-$Comp
-L NPN Q8
-U 1 1 54C48332
-P 7150 6550
-F 0 "Q8" H 7150 6400 50  0000 R CNN
-F 1 "NPN" H 7150 6700 50  0000 R CNN
-F 2 "~" H 7150 6550 60  0000 C CNN
-F 3 "~" H 7150 6550 60  0000 C CNN
-	1    7150 6550
 	0    1    1    0
 $EndComp
@@
 	1    9300 6400
 	1    0    0    -1
-$EndComp
-$Comp
-L NPN Q9
-U 1 1 54C48FF0
-P 10600 5750
-F 0 "Q9" H 10600 5600 50  0000 R CNN
-F 1 "NPN" H 10600 5900 50  0000 R CNN
-F 2 "~" H 10600 5750 60  0000 C CNN
-F 3 "~" H 10600 5750 60  0000 C CNN
-	1    10600 5750
-	0    1    -1   0
-$EndComp
-$Comp
-L NPN Q11
-U 1 1 54C48FFD
-P 11150 5850
-F 0 "Q11" H 11150 5700 50  0000 R CNN
-F 1 "NPN" H 11150 6000 50  0000 R CNN
-F 2 "~" H 11150 5850 60  0000 C CNN
-F 3 "~" H 11150 5850 60  0000 C CNN
-	1    11150 5850
-	0    1    -1   0
-$EndComp
-$Comp
-L NPN Q13
-U 1 1 54C4900A
-P 11700 5950
-F 0 "Q13" H 11700 5800 50  0000 R CNN
-F 1 "NPN" H 11700 6100 50  0000 R CNN
-F 2 "~" H 11700 5950 60  0000 C CNN
-F 3 "~" H 11700 5950 60  0000 C CNN
-	1    11700 5950
-	0    1    -1   0
-$EndComp
-$Comp
-L NPN Q15
-U 1 1 54C49017
-P 12250 6050
-F 0 "Q15" H 12250 5900 50  0000 R CNN
-F 1 "NPN" H 12250 6200 50  0000 R CNN
-F 2 "~" H 12250 6050 60  0000 C CNN
-F 3 "~" H 12250 6050 60  0000 C CNN
-	1    12250 6050
-	0    1    -1   0
-$EndComp
-$Comp
-L NPN Q10
-U 1 1 54C49024
-P 10600 6850
-F 0 "Q10" H 10600 6700 50  0000 R CNN
-F 1 "NPN" H 10600 7000 50  0000 R CNN
-F 2 "~" H 10600 6850 60  0000 C CNN
-F 3 "~" H 10600 6850 60  0000 C CNN
-	1    10600 6850
-	0    -1   1    0
-$EndComp
-$Comp
-L NPN Q12
-U 1 1 54C49031
-P 11150 6750
-F 0 "Q12" H 11150 6600 50  0000 R CNN
-F 1 "NPN" H 11150 6900 50  0000 R CNN
-F 2 "~" H 11150 6750 60  0000 C CNN
-F 3 "~" H 11150 6750 60  0000 C CNN
-	1    11150 6750
-	0    -1   1    0
-$EndComp
-$Comp
-L NPN Q14
-U 1 1 54C4903E
-P 11700 6650
-F 0 "Q14" H 11700 6500 50  0000 R CNN
-F 1 "NPN" H 11700 6800 50  0000 R CNN
-F 2 "~" H 11700 6650 60  0000 C CNN
-F 3 "~" H 11700 6650 60  0000 C CNN
-	1    11700 6650
-	0    -1   1    0
-$EndComp
-$Comp
-L NPN Q16
-U 1 1 54C4904B
-P 12250 6550
-F 0 "Q16" H 12250 6400 50  0000 R CNN
-F 1 "NPN" H 12250 6700 50  0000 R CNN
-F 2 "~" H 12250 6550 60  0000 C CNN
-F 3 "~" H 12250 6550 60  0000 C CNN
-	1    12250 6550
-	0    -1   1    0
 $EndComp
 Entry Wire Line
@@
 Text Label 3350 8100 0    30   ~ 0
 CLK
+$Comp
+L MMBT6427 Q1
+U 1 1 54C70802
+P 5500 5750
+F 0 "Q1" H 5500 5600 50  0000 R CNN
+F 1 "MMBT6427" H 5500 5900 50  0000 R CNN
+F 2 "~" H 5500 5750 60  0000 C CNN
+F 3 "~" H 5500 5750 60  0000 C CNN
+	1    5500 5750
+	0    -1   -1   0
+$EndComp
+$Comp
+L MMBT6427 Q3
+U 1 1 54C70822
+P 6050 5850
+F 0 "Q3" H 6050 5700 50  0000 R CNN
+F 1 "MMBT6427" H 6050 6000 50  0000 R CNN
+F 2 "~" H 6050 5850 60  0000 C CNN
+F 3 "~" H 6050 5850 60  0000 C CNN
+	1    6050 5850
+	0    -1   -1   0
+$EndComp
+$Comp
+L MMBT6427 Q5
+U 1 1 54C70831
+P 6600 5950
+F 0 "Q5" H 6600 5800 50  0000 R CNN
+F 1 "MMBT6427" H 6600 6100 50  0000 R CNN
+F 2 "~" H 6600 5950 60  0000 C CNN
+F 3 "~" H 6600 5950 60  0000 C CNN
+	1    6600 5950
+	0    -1   -1   0
+$EndComp
+$Comp
+L MMBT6427 Q7
+U 1 1 54C70840
+P 7150 6050
+F 0 "Q7" H 7150 5900 50  0000 R CNN
+F 1 "MMBT6427" H 7150 6200 50  0000 R CNN
+F 2 "~" H 7150 6050 60  0000 C CNN
+F 3 "~" H 7150 6050 60  0000 C CNN
+	1    7150 6050
+	0    -1   -1   0
+$EndComp
+$Comp
+L MMBT6427 Q8
+U 1 1 54C7084F
+P 7150 6550
+F 0 "Q8" H 7150 6400 50  0000 R CNN
+F 1 "MMBT6427" H 7150 6700 50  0000 R CNN
+F 2 "~" H 7150 6550 60  0000 C CNN
+F 3 "~" H 7150 6550 60  0000 C CNN
+	1    7150 6550
+	0    1    1    0
+$EndComp
+$Comp
+L MMBT6427 Q6
+U 1 1 54C7085E
+P 6600 6650
+F 0 "Q6" H 6600 6500 50  0000 R CNN
+F 1 "MMBT6427" H 6600 6800 50  0000 R CNN
+F 2 "~" H 6600 6650 60  0000 C CNN
+F 3 "~" H 6600 6650 60  0000 C CNN
+	1    6600 6650
+	0    1    1    0
+$EndComp
+$Comp
+L MMBT6427 Q4
+U 1 1 54C7086D
+P 6050 6750
+F 0 "Q4" H 6050 6600 50  0000 R CNN
+F 1 "MMBT6427" H 6050 6900 50  0000 R CNN
+F 2 "~" H 6050 6750 60  0000 C CNN
+F 3 "~" H 6050 6750 60  0000 C CNN
+	1    6050 6750
+	0    1    1    0
+$EndComp
+$Comp
+L MMBT6427 Q2
+U 1 1 54C7087C
+P 5500 6850
+F 0 "Q2" H 5500 6700 50  0000 R CNN
+F 1 "MMBT6427" H 5500 7000 50  0000 R CNN
+F 2 "~" H 5500 6850 60  0000 C CNN
+F 3 "~" H 5500 6850 60  0000 C CNN
+	1    5500 6850
+	0    -1   1    0
+$EndComp
+$Comp
+L MMBT6427 Q10
+U 1 1 54C70890
+P 10600 6850
+F 0 "Q10" H 10600 6700 50  0000 R CNN
+F 1 "MMBT6427" H 10600 7000 50  0000 R CNN
+F 2 "~" H 10600 6850 60  0000 C CNN
+F 3 "~" H 10600 6850 60  0000 C CNN
+	1    10600 6850
+	0    -1   1    0
+$EndComp
+$Comp
+L MMBT6427 Q12
+U 1 1 54C7089F
+P 11150 6750
+F 0 "Q12" H 11150 6600 50  0000 R CNN
+F 1 "MMBT6427" H 11150 6900 50  0000 R CNN
+F 2 "~" H 11150 6750 60  0000 C CNN
+F 3 "~" H 11150 6750 60  0000 C CNN
+	1    11150 6750
+	0    -1   1    0
+$EndComp
+$Comp
+L MMBT6427 Q14
+U 1 1 54C708AE
+P 11700 6650
+F 0 "Q14" H 11700 6500 50  0000 R CNN
+F 1 "MMBT6427" H 11700 6800 50  0000 R CNN
+F 2 "~" H 11700 6650 60  0000 C CNN
+F 3 "~" H 11700 6650 60  0000 C CNN
+	1    11700 6650
+	0    -1   1    0
+$EndComp
+$Comp
+L MMBT6427 Q16
+U 1 1 54C708BD
+P 12250 6550
+F 0 "Q16" H 12250 6400 50  0000 R CNN
+F 1 "MMBT6427" H 12250 6700 50  0000 R CNN
+F 2 "~" H 12250 6550 60  0000 C CNN
+F 3 "~" H 12250 6550 60  0000 C CNN
+	1    12250 6550
+	0    -1   1    0
+$EndComp
+$Comp
+L MMBT6427 Q15
+U 1 1 54C708CC
+P 12250 6050
+F 0 "Q15" H 12250 5900 50  0000 R CNN
+F 1 "MMBT6427" H 12250 6200 50  0000 R CNN
+F 2 "~" H 12250 6050 60  0000 C CNN
+F 3 "~" H 12250 6050 60  0000 C CNN
+	1    12250 6050
+	0    1    -1   0
+$EndComp
+$Comp
+L MMBT6427 Q13
+U 1 1 54C708DB
+P 11700 5950
+F 0 "Q13" H 11700 5800 50  0000 R CNN
+F 1 "MMBT6427" H 11700 6100 50  0000 R CNN
+F 2 "~" H 11700 5950 60  0000 C CNN
+F 3 "~" H 11700 5950 60  0000 C CNN
+	1    11700 5950
+	0    1    -1   0
+$EndComp
+$Comp
+L MMBT6427 Q11
+U 1 1 54C708EA
+P 11150 5850
+F 0 "Q11" H 11150 5700 50  0000 R CNN
+F 1 "MMBT6427" H 11150 6000 50  0000 R CNN
+F 2 "~" H 11150 5850 60  0000 C CNN
+F 3 "~" H 11150 5850 60  0000 C CNN
+	1    11150 5850
+	0    1    -1   0
+$EndComp
+$Comp
+L MMBT6427 Q9
+U 1 1 54C708FE
+P 10600 5750
+F 0 "Q9" H 10600 5600 50  0000 R CNN
+F 1 "MMBT6427" H 10600 5900 50  0000 R CNN
+F 2 "~" H 10600 5750 60  0000 C CNN
+F 3 "~" H 10600 5750 60  0000 C CNN
+	1    10600 5750
+	0    1    -1   0
+$EndComp
 $EndSCHEMATC

Commit message: Daily
Connections:
- net H is gone; now on net G: Q4.3 (C)
Changed lines of the file:
@@
 Sheet 1 1
 Title ""
-Date "27 jan 2015"
+Date "28 jan 2015"
 Rev ""
 Comp ""
@@
 $EndComp
 $Comp
-L GND #PWR9
+L GND #PWR01
 U 1 1 54C4804B
 P 5750 5650
-F 0 "#PWR9" H 5750 5650 30  0001 C CNN
+F 0 "#PWR01" H 5750 5650 30  0001 C CNN
 F 1 "GND" H 5750 5580 30  0001 C CNN
 F 2 "" H 5750 5650 60  0000 C CNN
@@
 $EndComp
 $Comp
-L GND #PWR11
+L GND #PWR02
 U 1 1 54C48233
 P 6300 5750
-F 0 "#PWR11" H 6300 5750 30  0001 C CNN
+F 0 "#PWR02" H 6300 5750 30  0001 C CNN
 F 1 "GND" H 6300 5680 30  0001 C CNN
 F 2 "" H 6300 5750 60  0000 C CNN
@@
 $EndComp
 $Comp
-L GND #PWR13
+L GND #PWR03
 U 1 1 54C48240
 P 6850 5850
-F 0 "#PWR13" H 6850 5850 30  0001 C CNN
+F 0 "#PWR03" H 6850 5850 30  0001 C CNN
 F 1 "GND" H 6850 5780 30  0001 C CNN
 F 2 "" H 6850 5850 60  0000 C CNN
@@
 $EndComp
 $Comp
-L GND #PWR15
+L GND #PWR04
 U 1 1 54C4824D
 P 7400 5950
-F 0 "#PWR15" H 7400 5950 30  0001 C CNN
+F 0 "#PWR04" H 7400 5950 30  0001 C CNN
 F 1 "GND" H 7400 5880 30  0001 C CNN
 F 2 "" H 7400 5950 60  0000 C CNN
@@
 $EndComp
 $Comp
-L GND #PWR10
+L GND #PWR05
 U 1 1 54C4831E
 P 5800 6850
-F 0 "#PWR10" H 5800 6850 30  0001 C CNN
+F 0 "#PWR05" H 5800 6850 30  0001 C CNN
 F 1 "GND" H 5800 6780 30  0001 C CNN
 F 2 "" H 5800 6850 60  0000 C CNN
@@
 $EndComp
 $Comp
-L GND #PWR12
+L GND #PWR06
 U 1 1 54C4832B
 P 6350 6750
-F 0 "#PWR12" H 6350 6750 30  0001 C CNN
+F 0 "#PWR06" H 6350 6750 30  0001 C CNN
 F 1 "GND" H 6350 6680 30  0001 C CNN
 F 2 "" H 6350 6750 60  0000 C CNN
@@
 $EndComp
 $Comp
-L GND #PWR14
+L GND #PWR07
 U 1 1 54C48338
 P 6900 6650
-F 0 "#PWR14" H 6900 6650 30  0001 C CNN
+F 0 "#PWR07" H 6900 6650 30  0001 C CNN
 F 1 "GND" H 6900 6580 30  0001 C CNN
 F 2 "" H 6900 6650 60  0000 C CNN
@@
 F
 Text Label 6250 7000 0    60   ~ 0
-H
+G
 Text Label 5700 7000 0    60   ~ 0
 9
@@
 8
 $Comp
-L VCC #PWR17
+L VCC #PWR08
 U 1 1 54C4907B
 P 10350 6950
-F 0 "#PWR17" H 10350 7050 30  0001 C CNN
+F 0 "#PWR08" H 10350 7050 30  0001 C CNN
 F 1 "VCC" H 10350 7050 30  0000 C CNN
 F 2 "" H 10350 6950 60  0000 C CNN
@@
 $EndComp
 $Comp
-L VCC #PWR19
+L VCC #PWR09
 U 1 1 54C490B7
 P 10900 6850
-F 0 "#PWR19" H 10900 6950 30  0001 C CNN
+F 0 "#PWR09" H 10900 6950 30  0001 C CNN
 F 1 "VCC" H 10900 6950 30  0000 C CNN
 F 2 "" H 10900 6850 60  0000 C CNN
@@
 $EndComp
 $Comp
-L VCC #PWR21
+L VCC #PWR010
 U 1 1 54C490C6
 P 11450 6750
-F 0 "#PWR21" H 11450 6850 30  0001 C CNN
+F 0 "#PWR010" H 11450 6850 30  0001 C CNN
 F 1 "VCC" H 11450 6850 30  0000 C CNN
 F 2 "" H 11450 6750 60  0000 C CNN
@@
 $EndComp
 $Comp
-L VCC #PWR23
+L VCC #PWR011
 U 1 1 54C490D5
 P 12000 6650
-F 0 "#PWR23" H 12000 6750 30  0001 C CNN
+F 0 "#PWR011" H 12000 6750 30  0001 C CNN
 F 1 "VCC" H 12000 6750 30  0000 C CNN
 F 2 "" H 12000 6650 60  0000 C CNN
@@
 $EndComp
 $Comp
-L VCC #PWR24
+L VCC #PWR012
 U 1 1 54C490E4
 P 12500 5950
-F 0 "#PWR24" H 12500 6050 30  0001 C CNN
+F 0 "#PWR012" H 12500 6050 30  0001 C CNN
 F 1 "VCC" H 12500 6050 30  0000 C CNN
 F 2 "" H 12500 5950 60  0000 C CNN
@@
 $EndComp
 $Comp
-L VCC #PWR22
+L VCC #PWR013
 U 1 1 54C490F3
 P 11950 5850
-F 0 "#PWR22" H 11950 5950 30  0001 C CNN
+F 0 "#PWR013" H 11950 5950 30  0001 C CNN
 F 1 "VCC" H 11950 5950 30  0000 C CNN
 F 2 "" H 11950 5850 60  0000 C CNN
@@
 $EndComp
 $Comp
-L VCC #PWR20
+L VCC #PWR014
 U 1 1 54C49102
 P 11400 5750
-F 0 "#PWR20" H 11400 5850 30  0001 C CNN
+F 0 "#PWR014" H 11400 5850 30  0001 C CNN
 F 1 "VCC" H 11400 5850 30  0000 C CNN
 F 2 "" H 11400 5750 60  0000 C CNN
@@
 $EndComp
 $Comp
-L VCC #PWR18
+L VCC #PWR015
 U 1 1 54C49111
 P 10850 5650
-F 0 "#PWR18" H 10850 5750 30  0001 C CNN
+F 0 "#PWR015" H 10850 5750 30  0001 C CNN
 F 1 "VCC" H 10850 5750 30  0000 C CNN
 F 2 "" H 10850 5650 60  0000 C CNN
@@
 9
 $Comp
-L VCC #PWR8
+L VCC #PWR016
 U 1 1 54C4A317
 P 5250 6950
-F 0 "#PWR8" H 5250 7050 30  0001 C CNN
+F 0 "#PWR016" H 5250 7050 30  0001 C CNN
 F 1 "VCC" H 5250 7050 30  0000 C CNN
 F 2 "" H 5250 6950 60  0000 C CNN
@@
 $EndComp
 $Comp
-L GND #PWR1
+L GND #PWR017
 U 1 1 54C589F6
 P 3700 8550
-F 0 "#PWR1" H 3700 8550 30  0001 C CNN
+F 0 "#PWR017" H 3700 8550 30  0001 C CNN
 F 1 "GND" H 3700 8480 30  0001 C CNN
 F 2 "" H 3700 8550 60  0000 C CNN
@@
 V3.3
 $Comp
-L GND #PWR3
+L GND #PWR018
 U 1 1 54C58D9C
 P 4200 9850
-F 0 "#PWR3" H 4200 9850 30  0001 C CNN
+F 0 "#PWR018" H 4200 9850 30  0001 C CNN
 F 1 "GND" H 4200 9780 30  0001 C CNN
 F 2 "" H 4200 9850 60  0000 C CNN
@@
 	3900 5650 3900 5850
 $Comp
-L GND #PWR2
+L GND #PWR019
 U 1 1 54C58F8A
 P 3900 7150
-F 0 "#PWR2" H 3900 7150 30  0001 C CNN
+F 0 "#PWR019" H 3900 7150 30  0001 C CNN
 F 1 "GND" H 3900 7080 30  0001 C CNN
 F 2 "" H 3900 7150 60  0000 C CNN
@@
 	3900 6950 3900 7150
 $Comp
-L GND #PWR16
+L GND #PWR020
 U 1 1 54C59085
 P 9000 7100
-F 0 "#PWR16" H 9000 7100 30  0001 C CNN
+F 0 "#PWR020" H 9000 7100 30  0001 C CNN
 F 1 "GND" H 9000 7030 30  0001 C CNN
 F 2 "" H 9000 7100 60  0000 C CNN
@@
 Connection ~ 3800 8400
 $Comp
-L VCC #PWR5
+L VCC #PWR021
 U 1 1 54C59360
 P 4600 8400
-F 0 "#PWR5" H 4600 8500 30  0001 C CNN
+F 0 "#PWR021" H 4600 8500 30  0001 C CNN
 F 1 "VCC" H 4600 8500 30  0000 C CNN
 F 2 "" H 4600 8400 60  0000 C CNN
@@
 $EndComp
 $Comp
-L GND #PWR4
+L GND #PWR022
 U 1 1 54C5937E
 P 4250 8950
-F 0 "#PWR4" H 4250 8950 30  0001 C CNN
+F 0 "#PWR022" H 4250 8950 30  0001 C CNN
 F 1 "GND" H 4250 8880 30  0001 C CNN
 F 2 "" H 4250 8950 60  0000 C CNN
@@
 $EndComp
 $Comp
-L GND #PWR6
+L GND #PWR023
 U 1 1 54C59633
 P 4700 10000
-F 0 "#PWR6" H 4700 10000 30  0001 C CNN
+F 0 "#PWR023" H 4700 10000 30  0001 C CNN
 F 1 "GND" H 4700 9930 30  0001 C CNN
 F 2 "" H 4700 10000 60  0000 C CNN
@@
 $EndComp
 $Comp
-L GND #PWR7
+L GND #PWR024
 U 1 1 54C5984D
 P 5200 10000
-F 0 "#PWR7" H 5200 10000 30  0001 C CNN
+F 0 "#PWR024" H 5200 10000 30  0001 C CNN
 F 1 "GND" H 5200 9930 30  0001 C CNN
 F 2 "" H 5200 10000 60  0000 C CNN
