File: TestDisplay/TestDisplay.kicad_pcb (KiCad board)
At the start: 2 copper layers, 111 parts, among them P1 CONN_6, Q1 MMBT6427, Q10 MMBT6427, Q11 MMBT6427, Q12 MMBT6427, Q13 MMBT6427, Q14 MMBT6427, Q15 MMBT6427, Q16 MMBT6427, Q2 MMBT6427, Q3 MMBT6427, Q4 MMBT6427, Q5 MMBT6427, Q6 MMBT6427, Q7 MMBT6427, Q8 MMBT6427, Q9 MMBT6427, U1 74LS595, U2 7805, U3 74LS595

Commit message: Daily
Parts:
- Q1, Q2: moved to F.Cu
- R10, R11, R12, R13, R14, R30, R31, R32, R33, R34, R35, R36, R37, R38, R39, R40, R41, R42, R43, R44, R45, R46, R47, R48, R49, R50, R66, R67, R68, R69, R70, R71, R72, R73, R74, R75, R76, R77, R78, R79, R9: moved to B.Cu
- moved R75 92.9 mm to (137.4, 99.3), turned to 270 degrees
- moved R74 90.2 mm to (140.0, 90.4), turned to 90 degrees
- moved R76 88.9 mm to (132.3, 99.3), turned to 270 degrees
- moved R73 88.0 mm to (137.4, 90.4), turned to 90 degrees
- moved R77 87.1 mm to (130.0, 99.3), turned to 270 degrees
- moved Q5 85.0 mm to (142.7, 71.5)
- moved R78 83.9 mm to (132.6, 90.4), turned to 90 degrees
- moved Q1 83.2 mm to (141.0, 50.5), turned to 90 degrees
- moved R79 81.8 mm to (130.0, 90.4), turned to 90 degrees
- moved Q4 80.5 mm to (141.0, 60.5), turned to 90 degrees
- moved Q3 79.5 mm to (141.0, 54.1), turned to 90 degrees
- moved U3 74.2 mm to (46.4, 69.0)
- moved R67 73.3 mm to (134.9, 53.1), turned to 90 degrees
- moved R68 72.4 mm to (132.3, 62.0), turned to 270 degrees
- moved R66 70.8 mm to (132.3, 53.1), turned to 90 degrees
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Connections:
- Q4 pad 3: (no net) -> /G
Routing:
- net /E: track 0.00 -> 184.7 mm, vias 0 -> 4
- net /F: track 0.00 -> 177.4 mm, vias 0 -> 4
- net /G: track 0.00 -> 173.4 mm, vias 0 -> 4
- net /D: track 0.00 -> 170.0 mm, vias 0 -> 4
- net /A: track 0.00 -> 169.2 mm, vias 0 -> 15
- net /B: track 0.00 -> 164.2 mm, vias 0 -> 13
- net /C: track 0.00 -> 159.7 mm, vias 0 -> 16
- net V3.3: track 58.5 -> 0.00 mm
- net /CLK: track 52.7 -> 0.00 mm, vias 2 -> 0
- net /STROBE: track 52.1 -> 0.00 mm, vias 2 -> 0
- net /DATA2: track 51.1 -> 0.00 mm
- net /DATA1: track 19.4 -> 0.00 mm
- net VCC: track 14.3 -> 0.00 mm
- net N-0000012: track 0.00 -> 2.62 mm
- net N-0000011: track 0.00 -> 2.60 mm
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
Commit message: Test Display Finished
Parts:
- C1, Q16, U2: moved to B.Cu
- R15, R16: moved to F.Cu
- moved Q6 82.4 mm to (141.0, 68.6), turned to 90 degrees
- moved Q8 81.4 mm to (141.0, 64.9), turned to 90 degrees
- moved R22 80.9 mm to (134.1, 81.7)
- moved Q7 80.6 mm to (141.0, 61.2), turned to 90 degrees
- moved R20 79.8 mm to (134.1, 79.2)
- moved R15 79.4 mm to (131.2, 73.0)
- moved R16 79.1 mm to (134.1, 74.3), turned to 0 degrees
- moved R18 78.8 mm to (134.1, 76.8)
- moved R21 77.7 mm to (131.2, 80.3)
- moved R19 76.6 mm to (131.2, 78.0)
- moved U1 76.3 mm to (121.7, 77.0)
- moved R17 75.6 mm to (131.2, 75.6)
- moved Q15 71.1 mm to (128.8, 69.3), turned to 90 degrees
- moved Q10 67.6 mm to (117.7, 83.2), turned to 270 degrees
- moved R61 67.5 mm to (124.6, 70.2)
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Connections:
- U2 pad 1: (no net) -> GND
- U2 pad 2: (no net) -> VCC
- U2 pad 3: (no net) -> V3.3
Routing:
- net GND: track 0.00 -> 316.7 mm, vias 0 -> 16
- net VCC: track 0.00 -> 171.7 mm, vias 0 -> 13
- net N-0000058: track 0.00 -> 110.3 mm
- net V3.3: track 0.00 -> 88.6 mm, vias 0 -> 5
- net /DATA1: track 0.00 -> 72.7 mm, vias 0 -> 1
- net /CLK: track 0.00 -> 68.6 mm, vias 0 -> 2
- net /STROBE: track 0.00 -> 67.2 mm, vias 0 -> 2
- net N-0000053: track 0.00 -> 54.1 mm
- net N-0000054: track 0.00 -> 53.4 mm, vias 0 -> 4
- net /F: track 177.4 -> 219.5 mm, vias 4 -> 7
- net N-0000059: track 0.00 -> 36.9 mm, vias 0 -> 2
- net /G: track 173.4 -> 209.6 mm, vias 4 -> 7
- net N-0000057: track 0.00 -> 31.0 mm
- net N-0000060: track 0.00 -> 29.9 mm
- net /DATA2: track 0.00 -> 29.3 mm, vias 0 -> 3
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- added copper zone on B.Cu, net GND
- added copper zone on F.Cu, net GND
Other:
- board outline added: 79 x 58.7 mm
- net class VCC added: clearance 0.254, trace_width 0.508, via_dia 1.016, via_drill 0.762
