File: TestDigit/Digit.kicad_pcb (KiCad board)
At the start: 2 copper layers, 100 x 100 mm, 95 parts, among them P1 CONN_6, P2 CONN_6, Q1 MMBT6427, Q10 MMBT6427, Q11 MMBT6427, Q12 MMBT6427, Q13 MMBT6427, Q14 MMBT6427, Q2 MMBT6427, Q3 MMBT6427, Q4 MMBT6427, Q5 MMBT6427, Q6 MMBT6427, Q7 MMBT6427, Q8 MMBT6427, Q9 MMBT6427, U1 74LS595, U2 74LS595

Commit message: Digit Fixes
Parts:
- moved D23 30.0 mm to (85.0, 120.0), turned to 90 degrees
- moved D29 30.0 mm to (85.0, 70.0), turned to 90 degrees
- moved D6 30.0 mm to (95.0, 70.0), turned to 90 degrees
- moved D36 20.0 mm to (125.0, 35.0), turned to 180 degrees
- moved D41 20.0 mm to (75.0, 80.0), turned to 180 degrees
- moved D42 20.0 mm to (125.0, 80.0), turned to 180 degrees
- moved D10 15.0 mm to (95.0, 105.0), turned to 90 degrees
- moved D19 15.0 mm to (85.0, 90.0), turned to 90 degrees
- moved D2 15.0 mm to (95.0, 40.0), turned to 90 degrees
- moved D20 15.0 mm to (135.0, 90.0), turned to 90 degrees
- moved D21 15.0 mm to (85.0, 105.0), turned to 90 degrees
- moved D22 15.0 mm to (135.0, 105.0), turned to 90 degrees
- moved D25 15.0 mm to (85.0, 40.0), turned to 90 degrees
- moved D26 15.0 mm to (135.0, 40.0), turned to 90 degrees
- moved D27 15.0 mm to (85.0, 55.0), turned to 90 degrees
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Connections:
- D1 pad 1: N-0000043 -> N-0000064
- D1 pad 2: N-0000044 -> N-0000063
- D10 pad 1: N-000005 (its old number) -> N-0000034
- D10 pad 2: N-000006 (its old number) -> N-0000047
- D11 pad 1: N-0000046 -> N-0000059
- D11 pad 2: N-0000047 -> N-0000016
- D12 pad 1: N-000005 (its old number) -> N-0000035
- D12 pad 2: N-000006 (its old number) -> N-0000034
- D13 pad 1: N-0000064 -> N-0000058
- D13 pad 2: N-0000062 -> N-0000060
- D14 pad 1: N-000003 -> N-0000037
- D14 pad 2: N-000004 -> N-0000036
- D15 pad 1: N-0000064 -> N-0000017
- D15 pad 2: N-0000062 -> N-0000058
- D16 pad 1: N-000003 -> N-0000020
- D16 pad 2: N-000004 -> N-0000037
- D17 pad 1: N-0000064 -> N-0000061
- D17 pad 2: N-0000062 -> N-0000017
- D18 pad 1: N-000003 -> N-0000038
- D18 pad 2: N-000004 -> N-0000020
- D19 pad 1: N-0000063 -> N-0000065
- D19 pad 2: N-0000054 -> N-0000062
- D2 pad 1: N-000007 (its old number) -> N-0000044
- D2 pad 2: N-000008 (its old number) -> N-0000043
- D20 pad 1: N-000002 -> N-0000040
- D20 pad 2: N-000001 (its old number) -> N-0000039
- D21 pad 1: N-0000063 -> N-0000018
- D21 pad 2: N-0000054 -> N-0000065
- D22 pad 1: N-000002 -> N-0000021
- D22 pad 2: N-000001 (its old number) -> N-0000040
- D23 pad 1: N-0000063 -> N-0000074
- D23 pad 2: N-0000054 -> N-0000018
- D24 pad 1: N-000002 -> N-0000054
- D24 pad 2: N-000001 (its old number) -> N-0000021
- D25 pad 1: N-0000066 -> N-0000075
- D25 pad 2: N-0000052 -> N-0000073
- D26 pad 1: N-0000011 (its old number) -> N-0000053
- D26 pad 2: N-0000012 (its old number) -> N-0000055
- D27 pad 1: N-0000066 -> N-0000019
- D27 pad 2: N-0000052 -> N-0000075
- D28 pad 1: N-0000011 (its old number) -> N-0000023
- D28 pad 2: N-0000012 (its old number) -> N-0000053
- D29 pad 1: N-0000066 -> N-0000076
- D29 pad 2: N-0000052 -> N-0000019
- D3 pad 1: N-0000043 -> N-000009
- D3 pad 2: N-0000044 -> N-0000064
- D30 pad 1: N-0000011 (its old number) -> N-0000056
- D30 pad 2: N-0000012 (its old number) -> N-0000023
- D31 pad 1: N-0000065 -> N-0000070
- D31 pad 2: N-0000042 -> N-0000069
- D32 pad 1: N-0000010 (its old number) -> N-0000049
- D32 pad 2: N-000009 -> N-0000057
- D33 pad 1: N-0000065 -> N-000003
- D33 pad 2: N-0000042 -> N-0000070
- D34 pad 1: N-0000010 (its old number) -> N-0000024
- D34 pad 2: N-000009 -> N-0000049
- D35 pad 1: N-0000065 -> N-0000068
- D35 pad 2: N-0000042 -> N-000003
- D36 pad 1: N-0000010 (its old number) -> N-0000050
- D36 pad 2: N-000009 -> N-0000024
- D37 pad 1: N-0000058 -> N-0000072
- D37 pad 2: N-0000040 -> N-0000071
- D38 pad 1: N-0000030 (its old number) -> N-0000051
- D38 pad 2: N-0000019 -> N-0000048
- D39 pad 1: N-0000058 -> N-000004
- D39 pad 2: N-0000040 -> N-0000072
- D4 pad 1: N-000007 (its old number) -> N-0000041
- D4 pad 2: N-000008 (its old number) -> N-0000044
- D40 pad 1: N-0000030 (its old number) -> N-0000025
- D40 pad 2: N-0000019 -> N-0000051
- D41 pad 1: N-0000058 -> N-0000042
- D41 pad 2: N-0000040 -> N-000004
- D42 pad 1: N-0000030 (its old number) -> N-0000052
- D42 pad 2: N-0000019 -> N-0000025
- D5 pad 1: N-0000043 -> N-0000066
- D5 pad 2: N-0000044 -> N-000009
- D6 pad 1: N-000007 (its old number) -> N-0000045
- D6 pad 2: N-000008 (its old number) -> N-0000041
- D7 pad 1: N-0000046 -> N-0000015
- D7 pad 2: N-0000047 -> N-0000067
- D8 pad 1: N-000005 (its old number) -> N-0000047
- D8 pad 2: N-000006 (its old number) -> N-0000046
- D9 pad 1: N-0000046 -> N-0000016
- D9 pad 2: N-0000047 -> N-0000015
- Q1 pad 3: N-0000044 -> N-0000063
- Q10 pad 3: N-0000012 (its old number) -> N-0000055
- Q11 pad 3: N-0000042 -> N-0000069
- Q12 pad 3: N-000009 -> N-0000057
- Q13 pad 3: N-0000040 -> N-0000071
- Q14 pad 3: N-0000019 -> N-0000048
- Q2 pad 3: N-000008 (its old number) -> N-0000043
- Q3 pad 3: N-0000047 -> N-0000067
- Q4 pad 3: N-000006 (its old number) -> N-0000046
- Q5 pad 3: N-0000062 -> N-0000060
- Q6 pad 3: N-000004 -> N-0000036
- Q7 pad 3: N-0000054 -> N-0000062
- Q8 pad 3: N-000001 (its old number) -> N-0000039
- Q9 pad 3: N-0000052 -> N-0000073
- R11 pad 2: N-0000064 -> N-0000061
- R12 pad 2: N-000003 -> N-0000038
- R15 pad 2: N-0000063 -> N-0000074
- R16 pad 2: N-000002 -> N-0000054
- R19 pad 2: N-0000066 -> N-0000076
- R20 pad 2: N-0000011 (its old number) -> N-0000056
- R23 pad 2: N-0000065 -> N-0000068
- R24 pad 2: N-0000010 (its old number) -> N-0000050
- R27 pad 2: N-0000058 -> N-0000042
- R28 pad 2: N-0000030 (its old number) -> N-0000052
- R3 pad 2: N-0000043 -> N-0000066
- R4 pad 2: N-000007 (its old number) -> N-0000045
- R7 pad 2: N-0000046 -> N-0000059
- R8 pad 2: N-000005 (its old number) -> N-0000035
Routing:
- net N-000008 (its old number): track 45.4 -> 0.00 mm
- net N-0000011 (its old number): track 37.1 -> 0.00 mm, vias 2 -> 0
- net N-000002: track 36.7 -> 0.00 mm, vias 2 -> 0
- net N-000006 (its old number): track 35.5 -> 0.00 mm, vias 2 -> 0
- net N-000005 (its old number): track 34.6 -> 0.00 mm
- net N-000007 (its old number): track 34.5 -> 0.00 mm
- net N-0000012 (its old number): track 33.8 -> 0.00 mm
- net N-000001 (its old number): track 32.9 -> 0.00 mm
- net N-0000044: track 45.5 -> 13.1 mm
- net N-0000058: track 36.1 -> 8.09 mm
- net N-0000030 (its old number): track 27.5 -> 0.00 mm, vias 2 -> 0
- net N-0000063: track 36.7 -> 10.7 mm, vias 2 -> 0
- net N-0000010 (its old number): track 24.6 -> 0.00 mm
- net N-0000047: track 36.9 -> 13.1 mm, vias 2 -> 0
- net N-0000046: track 34.7 -> 11.0 mm
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